Commit message: rotor inertia change + task integration

File: description/urdf/awesome_leg_complete_sliding.urdf (robot description, URDF)
Before this commit: robot awesome_leg_complete, 7 links, 6 joints
Joints:
- joint world_to_test_rig: axis (none) -> 0 1 0; type fixed -> prismatic

File: description/urdf/awesome_leg_fixed.xacro (robot description, xacro)
@@ -34,11 +34,8 @@
   </joint>
   <!-- Test rig to leg joint (prismatic); needs to be defined here since xbot2 cannot have passive joints in the URDF of the robot -->
-  <joint name="test_rig_pelvis" type="prismatic">
+  <joint name="test_rig_pelvis" type="fixed">
       <parent link="test_rig" />
       <child link="pelvis" />
-      <origin xyz="0 0 0.4" />
-      <axis xyz="0 0 1" />
-      <dynamics damping="0.0" friction="0.0" />
-      <limit lower="-0.8" upper="10.0" effort="80" velocity="15.0" />
+      <origin xyz="0 0 0.6" />
   </joint>
 </robot>

File: description/urdf/awesome_leg_sliding.xacro (robot description, xacro)
@@ -28,7 +28,8 @@
   <!--%%%%%%%%%%%%%%%% LOCALLY DEFINED JOINTS (not included through URDFs) %%%%%%%%%%%%%%%%-->
   <!-- fixing the test rig to the world -->
-  <joint name="world_test_rig" type="fixed">
+  <joint name="world_test_rig" type="prismatic">
         <parent link="world" />
         <child link="test_rig" />
+        <axis xyz="0 1 0" />
         <origin xyz="0 0 0.5" />
   </joint>
