Commit message: inertial parameters identification

File: description/urdf/awesome_leg_param_id.urdf (robot description, URDF)
Before this commit: robot awesome_leg, 5 links, 4 joints
Links:
- removed link hip1_1
- removed link hip2_1
- removed link knee_1
- removed link tip
- added link shank, mass 2.7264471; collision mesh filename=package://awesome_leg_pholus/description/meshes/collision/h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 scale=0.001 0.001 0.001; visual mesh filename=package://awesome_leg_pholus/description/meshes/visual/hip-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 scale=0.001 0.001 0.001
- added link shin, mass 1.23787877e+00; collision mesh filename=package://awesome_leg_pholus/description/meshes/collision/f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 scale=0.001 0.001 0.001; visual mesh filename=package://awesome_leg_pholus/description/meshes/visual/fron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 scale=0.001 0.001 0.001
Joints:
- removed joint base_joint
- removed joint hip_pitch_1
- removed joint knee_pitch_1
- removed joint tip_joint
- added joint hip_pitch: type revolute, parent world, child shank, origin xyz=0.0 0.0 0.0 rpy=-1.57 0 0, axis 0 0 1, limit lower=-2.0226 upper=2.02748 effort=112 velocity=20.0
- added joint knee_pitch: type revolute, parent shank, child shin, origin xyz=0.0 0.3 -0.0036 rpy=3.14159265359 0.0 1.57079632679, axis 0 0 1, limit lower=-2.0226 upper=2.02748 effort=112 velocity=20.0

File: description/urdf/awesome_leg_param_id_backup.urdf (robot description, URDF)
Before this commit: robot awesome_leg, 5 links, 4 joints
Links:
- removed link hip1_1
- removed link hip2_1
- removed link knee_1
- removed link tip
- added link shank, mass 2.7264471; collision mesh filename=package://awesome_leg_pholus/description/meshes/collision/h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 scale=0.001 0.001 0.001; visual mesh filename=package://awesome_leg_pholus/description/meshes/visual/hip-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 scale=0.001 0.001 0.001
- added link shin, mass 1.1927236; collision mesh filename=package://awesome_leg_pholus/description/meshes/collision/f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 scale=0.001 0.001 0.001; visual mesh filename=package://awesome_leg_pholus/description/meshes/visual/fron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 scale=0.001 0.001 0.001
Joints:
- removed joint base_joint
- removed joint hip_pitch_1
- removed joint knee_pitch_1
- removed joint tip_joint
- added joint hip_pitch: type revolute, parent world, child shank, origin xyz=0.0 0.0 0.0 rpy=-1.57 0 0, axis 0 0 1, limit lower=-2.0226 upper=2.02748 effort=112 velocity=20.0
- added joint knee_pitch: type revolute, parent shank, child shin, origin xyz=0.0 0.3 -0.0036 rpy=3.14159265359 0.0 1.57079632679, axis 0 0 1, limit lower=-2.0226 upper=2.02748 effort=112 velocity=20.0

Commit message: general improvs

File: description/urdf/awesome_leg_param_id.urdf (robot description, URDF)
Before this commit: robot awesome_leg, 3 links, 2 joints
Links:
- link shin: mass 1.23787877e+00 -> 1.1927236

Commit message: small changes

File: description/urdf/awesome_leg_param_id.urdf (robot description, URDF)
Before this commit: robot awesome_leg, 3 links, 2 joints
Joints:
- removed joint hip_pitch
- removed joint knee_pitch
- added joint hip_pitch_1: type revolute, parent world, child shank, origin xyz=0.0 0.0 0.0 rpy=-1.57 0 0, axis 0 0 1, limit lower=-2.0226 upper=2.02748 effort=112 velocity=20.0
- added joint knee_pitch_1: type revolute, parent shank, child shin, origin xyz=0.0 0.3 -0.0036 rpy=3.14159265359 0.0 1.57079632679, axis 0 0 1, limit lower=-2.0226 upper=2.02748 effort=112 velocity=20.0
