Commit message: fixed badly approximated values in URDF

File: description/urdf/awesome_leg_RBDL.urdf (robot description, URDF)
Before this commit: robot awesome_leg, 5 links, 4 joints
Joints:
- joint hip_pitch_1: origin xyz=0.0 0.0 0.0 rpy=-1.57 0 0 -> xyz=0.0 0.0 0.0 rpy=-1.57079632679 0 0

File: description/urdf/awesome_leg_reduced.urdf (robot description, URDF)
Before this commit: robot awesome_leg, 4 links, 3 joints
Joints:
- joint hip_pitch_1: origin xyz=0.0 0.0 0.0 rpy=-1.57 0 0 -> xyz=0.0 0.0 0.0 rpy=-1.57079632679 0 0

File: description/urdf/awesome_leg_reduced_calibrated.urdf (robot description, URDF)
Before this commit: robot awesome_leg, 4 links, 3 joints
Joints:
- joint hip_pitch_1: origin xyz=0.0 0.0 0.0 rpy=-1.57 0 0 -> xyz=0.0 0.0 0.0 rpy=-1.57079632679 0 0
