Commit message: small changes

File: description/urdf/awesome_leg_complete.urdf (robot description, URDF)
Before this commit: robot awesome_leg_complete, 7 links, 6 joints
Joints:
- removed joint test_rig_LF_HIP
- added joint passive_joint: type prismatic, parent test_rig, child pelvis, origin xyz=0 0 0.1, axis 0 0 1, limit lower=-0.5 upper=0.5 effort=80 velocity=15.0

Commit message: relative path integration fix

File: description/urdf/awesome_leg_complete.urdf (robot description, URDF)
Before this commit: robot awesome_leg_complete, 7 links, 6 joints
Joints:
- removed joint world_to_test_rig
- added joint world_test_rig: type fixed, parent world, child test_rig

File: description/urdf/awesome_leg_complete_fixed.urdf (robot description, URDF)
Before this commit: robot awesome_leg_complete, 7 links, 6 joints
Joints:
- removed joint world_to_test_rig
- added joint world_test_rig: type fixed, parent world, child test_rig

File: description/urdf/awesome_leg_complete_sliding_all.urdf (robot description, URDF)
Before this commit: robot awesome_leg_complete, 7 links, 6 joints
Joints:
- removed joint world_to_test_rig
- added joint world_test_rig: type prismatic, parent world, child test_rig, origin xyz=0 0 0.5, axis 0 1 0, limit lower=-100 upper=100.0 effort=1000000 velocity=100000000.0

File: description/urdf/awesome_leg_fixed.xacro (robot description, xacro)
@@ -34,5 +34,5 @@
   </joint>
   <!-- Test rig to leg joint (prismatic); needs to be defined here since xbot2 cannot have passive joints in the URDF of the robot -->
-  <joint name="test_rig_pelvis" type="fixed">
+  <joint name="passive_joint" type="fixed">
       <parent link="test_rig" />
       <child link="pelvis" />

File: description/urdf/awesome_leg_sliding_all.xacro (robot description, xacro)
@@ -37,5 +37,5 @@
   </joint>
   <!-- Test rig to leg joint (prismatic); needs to be defined here since xbot2 cannot have passive joints in the URDF of the robot -->
-  <joint name="test_rig_pelvis" type="prismatic">
+  <joint name="passive_joint" type="prismatic">
       <parent link="test_rig" />
       <child link="pelvis" />

Commit message: made knee_pitch_1 limits the same though all the URDF (xbot one was more conservative)

File: description/urdf/awesome_leg_complete.urdf (robot description, URDF)
Before this commit: robot awesome_leg_complete, 7 links, 6 joints
Joints:
- joint knee_pitch_1: limit lower=-2.4056 upper=2.3994 effort=112 velocity=20.0 -> lower=-2.0226 upper=2.02748 effort=112 velocity=20.0

File: description/urdf/awesome_leg_complete_fixed.urdf (robot description, URDF)
Before this commit: robot awesome_leg_complete_fixed, 7 links, 6 joints
Joints:
- joint knee_pitch_1: limit lower=-2.4056 upper=2.3994 effort=112 velocity=20.0 -> lower=-2.0226 upper=2.02748 effort=112 velocity=20.0
