Commit message: small changes

File: description/urdf/awesome_leg.xacro (robot description, xacro)
@@ -34,8 +34,8 @@
   </joint>
   <!-- Test rig to leg joint (prismatic); needs to be defined here since xbot2 cannot have passive joints in the URDF of the robot -->
-  <joint name="test_rig_LF_HIP" type="prismatic">
+  <joint name="test_rig_pelvis" type="prismatic">
       <parent link="test_rig" />
       <child link="pelvis" />
-      <origin xyz="0 0 0.1" />
+      <origin xyz="0 0 0.4" />
       <axis xyz="0 0 1" />
       <dynamics damping="0.0" friction="0.0" />

Commit message: current integration and plots

File: description/urdf/awesome_leg.xacro (robot description, xacro)
@@ -40,5 +40,5 @@
       <axis xyz="0 0 1" />
       <dynamics damping="0.0" friction="0.0" />
-      <limit lower="-0.5" upper="0.5" effort="80" velocity="15.0" />
+      <limit lower="-0.8" upper="0.5" effort="80" velocity="15.0" />
   </joint>
 </robot>

File: description/urdf/awesome_leg_complete.urdf (robot description, URDF)
Before this commit: robot awesome_leg_complete, 7 links, 6 joints
Joints:
- joint passive_joint: limit lower=-0.5 upper=0.5 effort=80 velocity=15.0 -> lower=-0.8 upper=0.5 effort=80 velocity=15.0

Commit message: general cleansing and relative path in YAML integration

File: description/urdf/awesome_leg.xacro (robot description, xacro)
@@ -13,5 +13,5 @@
               <box size="0.1 0.1 1" />
           </geometry>
-          <material name="test_rig_material" />
+          <material name="brown"/>
       </visual>
       <collision>
@@ -34,5 +34,5 @@
   </joint>
   <!-- Test rig to leg joint (prismatic); needs to be defined here since xbot2 cannot have passive joints in the URDF of the robot -->
-  <joint name="test_rig_pelvis" type="prismatic">
+  <joint name="passive_joint" type="prismatic">
       <parent link="test_rig" />
       <child link="pelvis" />

Commit message: removed comments from description files and small changes

File: description/urdf/awesome_leg.xacro (robot description, xacro)
@@ -2,5 +2,4 @@
 <robot name="awesome_leg" xmlns:xacro="http://www.ros.org/wiki/xacro">
   <!--%%%%%%%%%%%%%%%% CONSTANTS %%%%%%%%%%%%%%%%-->
-  <!--<xacro:property name="PI" value="3.1415926535897931"/> -->
   <!--%%%%%%%%%%%%%%%% IMPORTING ALL GAZEBO CUSTOMIZATION ELEMENTS %%%%%%%%%%%%%%%%-->
   <xacro:include filename="$(find awesome_leg_pholus)/description/urdf/awesome_leg.urdf" />

File: description/urdf/awesome_leg_cartesio.urdf (robot description, URDF)
Before this commit: robot awesome_leg, 5 links, 4 joints
Links:
- added link pelvis, mass 10.0; visual cylinder length=0.1 radius=0.1; visual cylinder length=0.1 radius=0.1
Joints:
- removed joint base_joint
- added joint 2world: type fixed, parent world, child pelvis
- added joint hip_yaw_1: type fixed, parent pelvis, child hip1_1, origin xyz=0.0 -0.0 -0.0566 rpy=3.14159265359 0.0 0.0
- joint hip_pitch_1: origin xyz=0.0 0.0 0.0 rpy=-1.57 0 0 -> xyz=0.0 0.0 0.0625 rpy=1.57079632679 0.0 1.5707963268

File: description/urdf/awesome_leg_fixed.xacro (robot description, xacro)
@@ -2,5 +2,4 @@
 <robot name="awesome_leg" xmlns:xacro="http://www.ros.org/wiki/xacro">
   <!--%%%%%%%%%%%%%%%% CONSTANTS %%%%%%%%%%%%%%%%-->
-  <!--<xacro:property name="PI" value="3.1415926535897931"/> -->
   <!--%%%%%%%%%%%%%%%% IMPORTING ALL GAZEBO CUSTOMIZATION ELEMENTS %%%%%%%%%%%%%%%%-->
   <xacro:include filename="$(find awesome_leg_pholus)/description/urdf/awesome_leg.urdf" />

File: description/urdf/awesome_leg_sliding_all.xacro (robot description, xacro)
@@ -2,5 +2,4 @@
 <robot name="awesome_leg" xmlns:xacro="http://www.ros.org/wiki/xacro">
   <!--%%%%%%%%%%%%%%%% CONSTANTS %%%%%%%%%%%%%%%%-->
-  <!--<xacro:property name="PI" value="3.1415926535897931"/> -->
   <!--%%%%%%%%%%%%%%%% IMPORTING ALL GAZEBO CUSTOMIZATION ELEMENTS %%%%%%%%%%%%%%%%-->
   <xacro:include filename="$(find awesome_leg_pholus)/description/urdf/awesome_leg.urdf" />

Commit message: added comments and improved repo organization

File: description/urdf/awesome_leg.xacro (robot description, xacro)
@@ -1,3 +1,6 @@
 <?xml version="1.0"?>
+<!--
+    Leg complete xacro with sliding hip. The main leg URDF is imported and the necessary links are added to it.
+-->
 <robot name="awesome_leg" xmlns:xacro="http://www.ros.org/wiki/xacro">
   <!--%%%%%%%%%%%%%%%% CONSTANTS %%%%%%%%%%%%%%%%-->

File: description/urdf/awesome_leg_RBDL.urdf (robot description, URDF)
Before this commit: robot awesome_leg, 4 links, 3 joints
Links:
- removed link shank
- removed link shin
- added link hip1_1, mass 1.9194403; collision mesh filename=package://awesome_leg_pholus/description/meshes/collision/h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 scale=0.001 0.001 0.001; visual mesh filename=package://awesome_leg_pholus/description/meshes/visual/hip-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 scale=0.001 0.001 0.001
- added link hip2_1, mass 2.7264471; collision mesh filename=package://awesome_leg_pholus/description/meshes/collision/h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 scale=0.001 0.001 0.001; visual mesh filename=package://awesome_leg_pholus/description/meshes/visual/hip-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 scale=0.001 0.001 0.001
- added link knee_1, mass 1.1927236; collision mesh filename=package://awesome_leg_pholus/description/meshes/collision/f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 scale=0.001 0.001 0.001; visual mesh filename=package://awesome_leg_pholus/description/meshes/visual/fron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 scale=0.001 0.001 0.001
Joints:
- added joint base_joint: type fixed, parent world, child hip1_1, origin xyz=0.0 -0.0 0.0 rpy=0.0 0.0 0.0
- joint hip_pitch_1: child shank -> hip2_1; parent world -> hip1_1
- joint knee_pitch_1: child shin -> knee_1; parent shank -> hip2_1
- joint tip_joint: parent shin -> knee_1

File: description/urdf/awesome_leg_fixed.xacro (robot description, xacro)
@@ -1,3 +1,6 @@
 <?xml version="1.0"?>
+<!--
+    Leg complete xacro with fixed hip. The main leg URDF is imported and the necessary links are added to it.
+-->
 <robot name="awesome_leg" xmlns:xacro="http://www.ros.org/wiki/xacro">
   <!--%%%%%%%%%%%%%%%% CONSTANTS %%%%%%%%%%%%%%%%-->

File: description/urdf/awesome_leg_reduced.urdf (robot description, URDF)
Before this commit: robot awesome_leg, 3 links, 2 joints
Links:
- added link tip
Joints:
- added joint tip_joint: type fixed, parent shin, child tip, origin xyz=0.45 0.0 -0.02

File: description/urdf/awesome_leg_reduced_calibrated.urdf (robot description, URDF)
Before this commit: robot awesome_leg, 5 links, 4 joints
Links:
- removed link hip1_1
- removed link hip2_1
- removed link knee_1
- added link shank, mass 2.7264471; collision mesh filename=package://awesome_leg_pholus/description/meshes/collision/h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 scale=0.001 0.001 0.001; visual mesh filename=package://awesome_leg_pholus/description/meshes/visual/hip-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 scale=0.001 0.001 0.001
- added link shin, mass 1.23787877e+00; collision mesh filename=package://awesome_leg_pholus/description/meshes/collision/f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 scale=0.001 0.001 0.001; visual mesh filename=package://awesome_leg_pholus/description/meshes/visual/fron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 scale=0.001 0.001 0.001
Joints:
- removed joint base_joint
- joint hip_pitch_1: child hip2_1 -> shank; parent hip1_1 -> world
- joint knee_pitch_1: child knee_1 -> shin; parent hip2_1 -> shank
- joint tip_joint: parent knee_1 -> shin

File: description/urdf/awesome_leg_sliding_all.xacro (robot description, xacro)
@@ -1,3 +1,6 @@
 <?xml version="1.0"?>
+<!--
+    Leg complete xacro with sliding hip and sliding test rig. The main leg URDF is imported and the necessary links are added to it.
+-->
 <robot name="awesome_leg" xmlns:xacro="http://www.ros.org/wiki/xacro">
   <!--%%%%%%%%%%%%%%%% CONSTANTS %%%%%%%%%%%%%%%%-->

Commit message: minor changes

File: description/urdf/awesome_leg.xacro (robot description, xacro)
@@ -42,5 +42,5 @@
       <axis xyz="0 0 1" />
       <dynamics damping="0.0" friction="0.0" />
-      <limit lower="-0.8" upper="10.0" effort="80" velocity="15.0" />
+      <limit lower="-10" upper="10.0" effort="500" velocity="50.0" />
   </joint>
 </robot>
