Commit message: pholus version

File: description/urdf/awesome_leg.urdf (robot description, URDF)
Before this commit: robot awesome_leg, 5 links, 4 joints
Links:
- removed link LF_ADAPTER
- removed link LF_FOOT
- removed link LF_HIP
- removed link LF_SHANK
- removed link LF_THIGH
- added link hip1_1, mass 1.9194403; collision mesh filename=package://awesome_leg_pholus/description/meshes/collision/h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 scale=0.001 0.001 0.001; visual mesh filename=package://awesome_leg_pholus/description/meshes/visual/hip-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 scale=0.001 0.001 0.001
- added link hip2_1, mass 2.7264471; collision mesh filename=package://awesome_leg_pholus/description/meshes/collision/h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 scale=0.001 0.001 0.001; visual mesh filename=package://awesome_leg_pholus/description/meshes/visual/hip-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 scale=0.001 0.001 0.001
- added link knee_1, mass 1.1927236; collision mesh filename=package://awesome_leg_pholus/description/meshes/collision/f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 scale=0.001 0.001 0.001; visual mesh filename=package://awesome_leg_pholus/description/meshes/visual/fron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 scale=0.001 0.001 0.001
- added link pelvis, mass 1.0; visual cylinder length=0.1 radius=0.1; visual cylinder length=0.1 radius=0.1
- added link tip
Joints:
- removed joint LF_ADAPTER_TO_FOOT
- removed joint LF_HFE
- removed joint LF_KFE
- removed joint LF_SHANK_TO_ADAPTER
- added joint hip_pitch_1: type revolute, parent hip1_1, child hip2_1, origin xyz=0.0 0.0 0.0625 rpy=1.57079632679 0.0 1.5707963268, axis 0 0 1, limit lower=-2.0226 upper=2.02748 effort=3040 velocity=28.8
- added joint hip_yaw_1: type fixed, parent pelvis, child hip1_1, origin xyz=0.0 -0.0 -0.0566 rpy=3.14159265359 0.0 0.0
- added joint knee_pitch_1: type revolute, parent hip2_1, child knee_1, origin xyz=0.0 0.3 -0.0036 rpy=3.14159265359 0.0 1.57079632679, axis 0 0 1, limit lower=-2.4056 upper=2.3994 effort=3040 velocity=28.8
- added joint tip_joint: type fixed, parent knee_1, child tip, origin xyz=0.45 0.0 -0.02

File: description/urdf/awesome_leg.xacro (robot description, xacro)
@@ -4,10 +4,10 @@
   <!--<xacro:property name="PI" value="3.1415926535897931"/> -->
   <!--%%%%%%%%%%%%%%%% IMPORTING ALL GAZEBO CUSTOMIZATION ELEMENTS %%%%%%%%%%%%%%%%-->
-  <xacro:include filename="$(find awesome_leg)/description/urdf/awesome_leg.urdf" />
+  <xacro:include filename="$(find awesome_leg_pholus)/description/urdf/awesome_leg.urdf" />
   <!--%%%%%%%%%%%%%%%% LOCALLY DEFINED LINKS (not included through URDFs) %%%%%%%%%%%%%%%%-->
   <link name="world" /> <!-- world link; necessary to make the test rig fixed -->
   <link name="test_rig"> <!-- test rig link; defined here to be able to cope with passive joints -->
       <visual>
-          <origin rpy="0 0 0" xyz="0.08 -0.13 0" />
+          <origin rpy="0 0 0" xyz="-0.12 0 0" />
           <geometry>
               <box size="0.1 0.1 1" />
@@ -16,5 +16,5 @@
       </visual>
       <collision>
-          <origin rpy="0 0 0" xyz="0.08 -0.13 0" />
+          <origin rpy="0 0 0" xyz="-0.12 0 0" />
           <geometry>
               <box size="0.1 0.1 1" />
@@ -36,5 +36,5 @@
   <joint name="test_rig_LF_HIP" type="prismatic">
       <parent link="test_rig" />
-      <child link="LF_HIP" />
+      <child link="pelvis" />
       <origin xyz="0 0 0.1" />
       <axis xyz="0 0 1" />

File: description/urdf/awesome_leg_complete.urdf (robot description, URDF)
Before this commit: robot awesome_leg_complete, 7 links, 6 joints
Links:
- removed link LF_ADAPTER
- removed link LF_FOOT
- removed link LF_HIP
- removed link LF_SHANK
- removed link LF_THIGH
- added link hip1_1, mass 1.9194403; collision mesh filename=package://awesome_leg_pholus/description/meshes/collision/h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 scale=0.001 0.001 0.001; visual mesh filename=package://awesome_leg_pholus/description/meshes/visual/hip-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 scale=0.001 0.001 0.001
- added link hip2_1, mass 2.7264471; collision mesh filename=package://awesome_leg_pholus/description/meshes/collision/h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 scale=0.001 0.001 0.001; visual mesh filename=package://awesome_leg_pholus/description/meshes/visual/hip-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 scale=0.001 0.001 0.001
- added link knee_1, mass 1.1927236; collision mesh filename=package://awesome_leg_pholus/description/meshes/collision/f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 scale=0.001 0.001 0.001; visual mesh filename=package://awesome_leg_pholus/description/meshes/visual/fron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 scale=0.001 0.001 0.001
- added link pelvis, mass 1.0; visual cylinder length=0.1 radius=0.1; visual cylinder length=0.1 radius=0.1
- added link tip
Joints:
- removed joint LF_ADAPTER_TO_FOOT
- removed joint LF_HFE
- removed joint LF_KFE
- removed joint LF_SHANK_TO_ADAPTER
- added joint hip_pitch_1: type revolute, parent hip1_1, child hip2_1, origin xyz=0.0 0.0 0.0625 rpy=1.57079632679 0.0 1.5707963268, axis 0 0 1, limit lower=-2.0226 upper=2.02748 effort=3040 velocity=28.8
- added joint hip_yaw_1: type fixed, parent pelvis, child hip1_1, origin xyz=0.0 -0.0 -0.0566 rpy=3.14159265359 0.0 0.0
- added joint knee_pitch_1: type revolute, parent hip2_1, child knee_1, origin xyz=0.0 0.3 -0.0036 rpy=3.14159265359 0.0 1.57079632679, axis 0 0 1, limit lower=-2.4056 upper=2.3994 effort=3040 velocity=28.8
- added joint tip_joint: type fixed, parent knee_1, child tip, origin xyz=0.45 0.0 -0.02
- joint test_rig_LF_HIP: child LF_HIP -> pelvis

Commit message: small changes

File: description/urdf/awesome_leg.urdf (robot description, URDF)
Before this commit: robot awesome_leg, 5 links, 4 joints
Links:
- link pelvis: mass 1.0 -> 10.0

File: description/urdf/awesome_leg_complete.urdf (robot description, URDF)
Before this commit: robot awesome_leg_complete, 7 links, 6 joints
Links:
- link pelvis: mass 1.0 -> 10.0

Commit message: gazebo simulation integration

File: description/urdf/awesome_leg.urdf (robot description, URDF)
Before this commit: robot awesome_leg, 5 links, 4 joints
Joints:
- joint hip_pitch_1: limit lower=-2.0226 upper=2.02748 effort=3040 velocity=28.8 -> lower=-2.0226 upper=2.02748 effort=100 velocity=30.0
- joint knee_pitch_1: limit lower=-2.4056 upper=2.3994 effort=3040 velocity=28.8 -> lower=-2.4056 upper=2.3994 effort=100 velocity=30.0

File: description/urdf/awesome_leg_complete.urdf (robot description, URDF)
Before this commit: robot awesome_leg_complete, 7 links, 6 joints
Joints:
- joint hip_pitch_1: limit lower=-2.0226 upper=2.02748 effort=3040 velocity=28.8 -> lower=-2.0226 upper=2.02748 effort=100 velocity=35.0
- joint knee_pitch_1: limit lower=-2.4056 upper=2.3994 effort=3040 velocity=28.8 -> lower=-2.4056 upper=2.3994 effort=100 velocity=35.0

Commit message: actuators test integration

File: description/urdf/awesome_leg.urdf (robot description, URDF)
Before this commit: robot awesome_leg, 5 links, 4 joints
Joints:
- joint hip_pitch_1: limit lower=-2.0226 upper=2.02748 effort=100 velocity=30.0 -> lower=-2.0226 upper=2.02748 effort=112 velocity=20.0
- joint knee_pitch_1: limit lower=-2.4056 upper=2.3994 effort=100 velocity=30.0 -> lower=-2.4056 upper=2.3994 effort=112 velocity=20.0

File: description/urdf/awesome_leg_complete.urdf (robot description, URDF)
Before this commit: robot awesome_leg_complete, 7 links, 6 joints
Joints:
- joint hip_pitch_1: limit lower=-2.0226 upper=2.02748 effort=100 velocity=35.0 -> lower=-2.0226 upper=2.02748 effort=112 velocity=20.0
- joint knee_pitch_1: limit lower=-2.4056 upper=2.3994 effort=100 velocity=35.0 -> lower=-2.4056 upper=2.3994 effort=112 velocity=20.0

Commit message: leg visual improvs

File: description/urdf/awesome_leg.urdf (robot description, URDF)
Before this commit: robot awesome_leg, 5 links, 4 joints
Joints:
- joint knee_pitch_1: limit lower=-2.4056 upper=2.3994 effort=112 velocity=20.0 -> lower=-2.0226 upper=2.02748 effort=112 velocity=20.0

File: description/urdf/awesome_leg_fixed.xacro (robot description, xacro)
@@ -13,5 +13,5 @@
               <box size="0.1 0.1 1" />
           </geometry>
-          <material name="test_rig_material" />
+          <material name="brown" />
       </visual>
       <collision>

File: description/urdf/awesome_leg_sliding_all.xacro (robot description, xacro)
@@ -13,5 +13,5 @@
               <box size="0.1 0.1 1" />
           </geometry>
-          <material name="test_rig_material" />
+          <material name="brown" />
       </visual>
       <collision>

Commit message: general restyling and jump opt improvements and tuning

File: description/urdf/awesome_leg.urdf (robot description, URDF)
Before this commit: robot awesome_leg, 5 links, 4 joints
Links:
- link pelvis: mass 10.0 -> 1.0

File: description/urdf/awesome_leg_complete.urdf (robot description, URDF)
Before this commit: robot awesome_leg_complete, 7 links, 6 joints
Links:
- link pelvis: mass 10.0 -> 1.0
Joints:
- joint passive_joint: limit lower=-0.8 upper=10.0 effort=80 velocity=15.0 -> lower=-1 upper=1.0 effort=80 velocity=15.0

Commit message: modified ros package name

File: description/urdf/awesome_leg.urdf (robot description, URDF)
Before this commit: robot awesome_leg, 5 links, 4 joints
Links:
- link hip1_1: geometry collision mesh filename=package://awesome_leg/description/meshes/collision/hip-yaw.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 scale=0.001 0.001 0.001; visual mesh filename=package://awesome_leg/description/meshes/visual/hip-yaw.stl scale=0.001 0.001 0.001
- link hip2_1: geometry collision mesh filename=package://awesome_leg/description/meshes/collision/hip-pitc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 scale=0.001 0.001 0.001; visual mesh filename=package://awesome_leg/description/meshes/visual/hip-pitch.s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 scale=0.001 0.001 0.001
- link knee_1: geometry collision mesh filename=package://awesome_leg/description/meshes/collision/front_ri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 scale=0.001 0.001 0.001; visual mesh filename=package://awesome_leg/description/meshes/visual/front_right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 scale=0.001 0.001 0.001

File: description/urdf/awesome_leg.xacro (robot description, xacro)
@@ -6,5 +6,5 @@
   <!--%%%%%%%%%%%%%%%% CONSTANTS %%%%%%%%%%%%%%%%-->
   <!--%%%%%%%%%%%%%%%% IMPORTING ALL GAZEBO CUSTOMIZATION ELEMENTS %%%%%%%%%%%%%%%%-->
-  <xacro:include filename="$(find awesome_leg_pholus)/description/urdf/awesome_leg.urdf" />
+  <xacro:include filename="$(find awesome_leg)/description/urdf/awesome_leg.urdf" />
   <!--%%%%%%%%%%%%%%%% LOCALLY DEFINED LINKS (not included through URDFs) %%%%%%%%%%%%%%%%-->
   <link name="world" /> <!-- world link; necessary to make the test rig fixed -->

File: description/urdf/awesome_leg_RBDL.urdf (robot description, URDF)
Before this commit: robot awesome_leg, 5 links, 4 joints
Links:
- link hip1_1: geometry collision mesh filename=package://awesome_leg/description/meshes/collision/hip-yaw.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 scale=0.001 0.001 0.001; visual mesh filename=package://awesome_leg/description/meshes/visual/hip-yaw.stl scale=0.001 0.001 0.001
- link hip2_1: geometry collision mesh filename=package://awesome_leg/description/meshes/collision/hip-pitc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 scale=0.001 0.001 0.001; visual mesh filename=package://awesome_leg/description/meshes/visual/hip-pitch.s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 scale=0.001 0.001 0.001
- link knee_1: geometry collision mesh filename=package://awesome_leg/description/meshes/collision/front_ri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 scale=0.001 0.001 0.001; visual mesh filename=package://awesome_leg/description/meshes/visual/front_right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 scale=0.001 0.001 0.001

File: description/urdf/awesome_leg_cartesio.urdf (robot description, URDF)
Before this commit: robot awesome_leg, 6 links, 5 joints
Links:
- link hip1_1: geometry collision mesh filename=package://awesome_leg/description/meshes/collision/hip-yaw.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 scale=0.001 0.001 0.001; visual mesh filename=package://awesome_leg/description/meshes/visual/hip-yaw.stl scale=0.001 0.001 0.001
- link hip2_1: geometry collision mesh filename=package://awesome_leg/description/meshes/collision/hip-pitc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 scale=0.001 0.001 0.001; visual mesh filename=package://awesome_leg/description/meshes/visual/hip-pitch.s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 scale=0.001 0.001 0.001
- link knee_1: geometry collision mesh filename=package://awesome_leg/description/meshes/collision/front_ri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 scale=0.001 0.001 0.001; visual mesh filename=package://awesome_leg/description/meshes/visual/front_right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 scale=0.001 0.001 0.001

File: description/urdf/awesome_leg_complete.urdf (robot description, URDF)
Before this commit: robot awesome_leg_complete, 7 links, 6 joints
Links:
- link hip1_1: geometry collision mesh filename=package://awesome_leg/description/meshes/collision/hip-yaw.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 scale=0.001 0.001 0.001; visual mesh filename=package://awesome_leg/description/meshes/visual/hip-yaw.stl scale=0.001 0.001 0.001
- link hip2_1: geometry collision mesh filename=package://awesome_leg/description/meshes/collision/hip-pitc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 scale=0.001 0.001 0.001; visual mesh filename=package://awesome_leg/description/meshes/visual/hip-pitch.s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 scale=0.001 0.001 0.001
- link knee_1: geometry collision mesh filename=package://awesome_leg/description/meshes/collision/front_ri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 scale=0.001 0.001 0.001; visual mesh filename=package://awesome_leg/description/meshes/visual/front_right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 scale=0.001 0.001 0.001

File: description/urdf/awesome_leg_complete_fixed.urdf (robot description, URDF)
Before this commit: robot awesome_leg_complete_fixed, 7 links, 6 joints
Links:
- link hip1_1: geometry collision mesh filename=package://awesome_leg/description/meshes/collision/hip-yaw.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 scale=0.001 0.001 0.001; visual mesh filename=package://awesome_leg/description/meshes/visual/hip-yaw.stl scale=0.001 0.001 0.001
- link hip2_1: geometry collision mesh filename=package://awesome_leg/description/meshes/collision/hip-pitc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 scale=0.001 0.001 0.001; visual mesh filename=package://awesome_leg/description/meshes/visual/hip-pitch.s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 scale=0.001 0.001 0.001
- link knee_1: geometry collision mesh filename=package://awesome_leg/description/meshes/collision/front_ri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 scale=0.001 0.001 0.001; visual mesh filename=package://awesome_leg/description/meshes/visual/front_right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 scale=0.001 0.001 0.001

File: description/urdf/awesome_leg_fixed.xacro (robot description, xacro)
@@ -6,5 +6,5 @@
   <!--%%%%%%%%%%%%%%%% CONSTANTS %%%%%%%%%%%%%%%%-->
   <!--%%%%%%%%%%%%%%%% IMPORTING ALL GAZEBO CUSTOMIZATION ELEMENTS %%%%%%%%%%%%%%%%-->
-  <xacro:include filename="$(find awesome_leg_pholus)/description/urdf/awesome_leg.urdf" />
+  <xacro:include filename="$(find awesome_leg)/description/urdf/awesome_leg.urdf" />
   <!--%%%%%%%%%%%%%%%% LOCALLY DEFINED LINKS (not included through URDFs) %%%%%%%%%%%%%%%%-->
   <link name="world" /> <!-- world link; necessary to make the test rig fixed -->

File: description/urdf/awesome_leg_original.urdf (robot description, URDF)
Before this commit: robot awesome_leg, 5 links, 4 joints
Links:
- link hip1_1: geometry collision mesh filename=package://awesome_leg/description/meshes/collision/hip-yaw.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 scale=0.001 0.001 0.001; visual mesh filename=package://awesome_leg/description/meshes/visual/hip-yaw.stl scale=0.001 0.001 0.001
- link hip2_1: geometry collision mesh filename=package://awesome_leg/description/meshes/collision/hip-pitc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 scale=0.001 0.001 0.001; visual mesh filename=package://awesome_leg/description/meshes/visual/hip-pitch.s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 scale=0.001 0.001 0.001
- link knee_1: geometry collision mesh filename=package://awesome_leg/description/meshes/collision/front_ri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 scale=0.001 0.001 0.001; visual mesh filename=package://awesome_leg/description/meshes/visual/front_right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 scale=0.001 0.001 0.001

File: description/urdf/awesome_leg_reduced.urdf (robot description, URDF)
Before this commit: robot awesome_leg, 4 links, 3 joints
Links:
- link shank: geometry collision mesh filename=package://awesome_leg/description/meshes/collision/hip-pitc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 scale=0.001 0.001 0.001; visual mesh filename=package://awesome_leg/description/meshes/visual/hip-pitch.s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 scale=0.001 0.001 0.001
- link shin: geometry collision mesh filename=package://awesome_leg/description/meshes/collision/front_ri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 scale=0.001 0.001 0.001; visual mesh filename=package://awesome_leg/description/meshes/visual/front_right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 scale=0.001 0.001 0.001

File: description/urdf/awesome_leg_reduced_calibrated.urdf (robot description, URDF)
Before this commit: robot awesome_leg, 4 links, 3 joints
Links:
- link shank: geometry collision mesh filename=package://awesome_leg/description/meshes/collision/hip-pitc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 scale=0.001 0.001 0.001; visual mesh filename=package://awesome_leg/description/meshes/visual/hip-pitch.s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 scale=0.001 0.001 0.001
- link shin: geometry collision mesh filename=package://awesome_leg/description/meshes/collision/front_ri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 scale=0.001 0.001 0.001; visual mesh filename=package://awesome_leg/description/meshes/visual/front_right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 scale=0.001 0.001 0.001

File: description/urdf/awesome_leg_sliding_all.xacro (robot description, xacro)
@@ -6,5 +6,5 @@
   <!--%%%%%%%%%%%%%%%% CONSTANTS %%%%%%%%%%%%%%%%-->
   <!--%%%%%%%%%%%%%%%% IMPORTING ALL GAZEBO CUSTOMIZATION ELEMENTS %%%%%%%%%%%%%%%%-->
-  <xacro:include filename="$(find awesome_leg_pholus)/description/urdf/awesome_leg.urdf" />
+  <xacro:include filename="$(find awesome_leg)/description/urdf/awesome_leg.urdf" />
   <!--%%%%%%%%%%%%%%%% LOCALLY DEFINED LINKS (not included through URDFs) %%%%%%%%%%%%%%%%-->
   <link name="world" /> <!-- world link; necessary to make the test rig fixed -->
