Commit message: minor changes

File: description/urdf/awesome_leg_original.urdf (robot description, URDF)
Before this commit: robot awesome_leg, 5 links, 4 joints
Links:
- link pelvis: mass 10.0 -> 1.0

Commit message: description file cutdown and other improvements

File: description/urdf/awesome_leg_original.urdf (robot description, URDF)
Before this commit: robot awesome_leg, 5 links, 4 joints
Links:
- added link base_link, mass 1.0; collision box size=0.1 0.1 1.5; visual box size=0.1 0.1 1.5
- added link world
- link hip1_1: geometry collision mesh filename=package://centauro_urdf/meshes/simple/hip-yaw.stl scale=0.001 0.001 0.001; visual mesh filename=package://centauro_urdf/meshes/hip-yaw.stl scale=0.001 0.001 0.001
- link hip2_1: geometry collision mesh filename=package://centauro_urdf/meshes/simple/hip-pitch.stl scale=0.001 0.001 0.001; visual mesh filename=package://centauro_urdf/meshes/hip-pitch.stl scale=0.001 0.001 0.001
- link knee_1: geometry collision mesh filename=package://centauro_urdf/meshes/simple/front_right_stick.stl scale=0.001 0.001 0.001; visual mesh filename=package://centauro_urdf/meshes/front_right_stick.stl scale=0.001 0.001 0.001
Joints:
- added joint passive_joint: type prismatic, parent base_link, child pelvis, origin xyz=0.15 0. 0.8, axis 0 0 1, limit lower=-3.5 upper=3.5 effort=1000.0 velocity=100.
- added joint reference: type fixed, parent world, child base_link, origin xyz=0 0 0 rpy=0 0 0
- joint hip_pitch_1: limit lower=-2.0226 upper=2.02748 effort=112 velocity=20.0 -> lower=-2.0226 upper=2.02748 effort=3040 velocity=28.8
- joint knee_pitch_1: limit lower=-2.0226 upper=2.02748 effort=112 velocity=20.0 -> lower=-2.4056 upper=2.3994 effort=3040 velocity=28.8
