Commit message: added compensation for wrong metal plate weight

File: description/urdf/utils.urdf.xacro (robot description, xacro)
@@ -11,5 +11,6 @@
 <xacro:property name="PI_4" value="0.7853981633974483" />
 <xacro:property name="DEG2RAD" value="${PI/180.0}" />
-<xacro:property name="payload_mass" value="0.0" />
+<xacro:property name="base_link_mass_compensation" value="2.0" />
+<xacro:property name="payload_mass" value="${0.0 + base_link_mass_compensation}" />
 <!-- <xacro:property name="payload_mass" value="7.38" /> -->
 <xacro:property name="camera_height" value="0.5" />

Commit message: removed friction on linear guide

File: description/urdf/utils.urdf.xacro (robot description, xacro)
@@ -12,5 +12,6 @@
 <xacro:property name="DEG2RAD" value="${PI/180.0}" />
 <xacro:property name="sliding_guide_static_friction" value="0.0" />
-<xacro:property name="sliding_guide_dyn_friction" value="50.0" />
+<xacro:property name="sliding_guide_dyn_friction" value="0.0" />
+<!--<xacro:property name="sliding_guide_dyn_friction" value="50.0" />-->
 <xacro:property name="base_link_mass_compensation" value="2.0" />
 <xacro:property name="payload_mass" value="${0.0 + base_link_mass_compensation}" />
