Commit message: new meshes and inertial paramters integration into URDFs

File: description/urdf/awesome_leg.gazebo.xacro (robot description, xacro)
@@ -1,32 +1,41 @@
 <?xml version="1.0"?>
 <robot xmlns:xacro="http://ros.org/wiki/xacro">
-<gazebo reference="knee_1">
-    <collision>
-        <surface>
-            <friction>
-                <ode>
-                    <mu>1.0</mu>
-                    <mu2>1.0</mu2>
-                </ode>
-                <bullet>
-                    <friction>1.0</friction>
-                    <friction2>1.0</friction2>
-                </bullet>
-            </friction>
-            <contact>
-                <ode>
-                    <kp>2100000</kp>
-                    <kd>1</kd>
-                    <max_vel>100</max_vel>
-                </ode>
-                <bullet>
-                    <soft_cfm>0.007</soft_cfm>
-                    <soft_erp>0.25</soft_erp>
-                    <kp>1000000</kp>
-                    <kd>5</kd>
-                </bullet>
-            </contact>
-        </surface>
-    </collision>
-</gazebo>
+    <xacro:macro name="awesome_leg" params="id" >
+    <!--Gazebo-specific tags-->
+        <gazebo reference="femur${id}">
+            <material>Gazebo/SkyBlue  </material>
+        </gazebo>
+        <gazebo reference="shin${id}">
+            <material>Gazebo/Grey  </material>
+        </gazebo>
+        <!-- <gazebo reference="knee_1">
+            <collision>
+                <surface>
+                    <friction>
+                        <ode>
+                            <mu>1.0</mu>
+                            <mu2>1.0</mu2>
+                        </ode>
+                        <bullet>
+                            <friction>1.0</friction>
+                            <friction2>1.0</friction2>
+                        </bullet>
+                    </friction>
+                    <contact>
+                        <ode>
+                            <kp>2100000</kp>
+                            <kd>1</kd>
+                            <max_vel>100</max_vel>
+                        </ode>
+                        <bullet>
+                            <soft_cfm>0.007</soft_cfm>
+                            <soft_erp>0.25</soft_erp>
+                            <kp>1000000</kp>
+                            <kd>5</kd>
+                        </bullet>
+                    </contact>
+                </surface>
+            </collision>
+        </gazebo> -->
+    </xacro:macro>
 </robot>

File: description/urdf/awesome_leg.urdf.xacro (robot description, xacro)
@@ -1,157 +1,91 @@
 <?xml version="1.0" encoding="utf-8" ?>
 <robot name="awesome_leg" xmlns:xacro="http://www.ros.org/wiki/xacro">
-    <xacro:include filename="$(find awesome_leg)/description/urdf/utils.urdf.xacro" />
     <xacro:include filename="$(find awesome_leg)/description/urdf/awesome_leg.gazebo.xacro" />
-    <link name="pelvis">
-        <inertial>
-        <mass value="1.0"/> <!-- here an additional mass contribution can be added to mimic a weight can be added (standard link mass = 1 Kg) -->
-        <inertia ixx="0.00208333333333" ixy="0.0" ixz="0.0" iyy="0.00208333333333" iyz="0.0" izz="0.0025"/>
-        </inertial>
-        <visual>
-        <geometry>
-            <cylinder length="0.1" radius="0.1"/>
-        </geometry>
-        </visual>
-        <visual>
-        <geometry>
-            <cylinder length="0.1" radius="0.1"/>
-        </geometry>
-        </visual>
-    </link>
-    <joint name="hip_yaw_1" type="fixed">
-        <parent link="pelvis"/>
-        <child link="hip1_1"/>
-        <origin rpy="3.14159265359 0.0 0.0" xyz="0.0 -0.0 -0.0566"/>
-    </joint>
-    <link name="hip1_1">
-        <inertial>
-        <origin xyz="0.010214199 0.0 0.038090987"/>
-        <mass value="1.9194403"/>
-        <inertia ixx="0.0047439572" ixy="-0.0" ixz="-0.0003784138" iyy="0.0040551878" iyz="-0.0" izz="0.0034146219"/>
-        </inertial>
-        <visual>
-        <origin rpy="0.0 0.0 2.03221245002" xyz="0.0 0.0 0.0"/>
-        <geometry>
-            <mesh filename="package://awesome_leg/description/meshes/visual/hip-yaw.stl" scale="0.001 0.001 0.001"/>
-        </geometry>
-        <material name="grey"/>
-        </visual>
-        <collision>
-        <origin rpy="0.0 0.0 2.03221245002" xyz="0.0 0.0 0.0"/>
-        <geometry>
-            <mesh filename="package://awesome_leg/description/meshes/collision/hip-yaw.stl" scale="0.001 0.001 0.001"/>
-        </geometry>
-        </collision>
-    </link>
-    <joint name="hip_pitch_1" type="revolute">
-        <parent link="hip1_1"/>
-        <child link="hip2_1"/>
-        <origin rpy="1.57079632679 0.0 1.5707963268" xyz="0.0 0.0 0.0625"/>
-        <axis xyz="0 0 1"/>
-        <limit effort="112" lower="-2.4" upper="2.4" velocity="20.0"/>
-    </joint>
-    <link name="hip2_1"> <!-- #### -->
-        <inertial>
-        <origin xyz="2.57966e-05 0.1810266 0.085669756"/>
-        <mass value="2.7264471"/>
-        <!-- org: 4.5 -->
-        <inertia ixx="0.04851869" ixy="-4.11894e-05" ixz="-1.68778e-05" iyy="0.004242055" iyz="0.0032243188" izz="0.04825583"/>
-        </inertial>
-        <visual>
-        <origin rpy="0.0 0.0 0.0" xyz="0.0 0.0 0.0"/>
-        <material name="sky_blue"/>
-        <geometry>
-            <mesh filename="package://awesome_leg/description/meshes/visual/hip-pitch.stl" scale="0.001 0.001 0.001"/>
-        </geometry>
-        </visual>
-        <collision>
-        <origin rpy="0.0 0.0 0.0" xyz="0.0 0.0 0.0"/>
-        <geometry>
-            <mesh filename="package://awesome_leg/description/meshes/collision/hip-pitch.stl" scale="0.001 0.001 0.001"/>
-        </geometry>
-        </collision>
-    </link>
-    <joint name="knee_pitch_1" type="revolute">
-        <parent link="hip2_1"/>
-        <child link="knee_1"/>
-        <origin rpy="3.14159265359 0.0 1.57079632679" xyz="0.0 0.3 -0.0036"/>
-        <axis xyz="0 0 1"/>grey
-        <limit effort="112" lower="-2.4" upper="2.4" velocity="20.0"/>
-    </joint>
-    <link name="knee_1"> <!-- #### -->
-        <inertial>
-        <mass value="1.1927236"/>
-        <origin rpy="0.0 0.0 0.0" xyz="0.19572282 -0.014549221 -0.020785942"/>
-        <inertia ixx="0.0013302597" ixy="0.00060307457" ixz="0.0" iyy="0.035313402" iyz="-1.1029574e-07" izz="0.035530025"/>
-        </inertial>
-        <visual>
-        <origin rpy="1.57079632679 0 -1.57079632679" xyz="0 0 0"/>
-        <material name="grey"/>
-        <geometry name="1_stick_visual">
-            <mesh filename="package://awesome_leg/description/meshes/visual/front_right_stick.stl" scale="0.001 0.001 0.001"/>
-        </geometry>
-        </visual>
-        <collision name="foot_tip_collision">
-        <origin rpy="1.57079632679 0 -1.57079632679" xyz="0 0 0"/>
-        <geometry name="1_stick_collision">
-            <mesh filename="package://awesome_leg/description/meshes/collision/front_right_stick.stl" scale="0.001 0.001 0.001"/>
-        </geometry>
-        </collision>
-    </link>
-    <joint name="tip_joint" type="fixed">
-        <parent link="knee_1"/>
-        <child link="tip"/>
-        <origin xyz="0.45 0.0 -0.02"/>
-    </joint>
-    <link name="tip"/> <!-- just for reference-->
-    <transmission name="hip_trans">
-        <type>transmission_interface/SimpleTransmission</type>
-        <joint name="hip_pitch_1">
-            <hardwareInterface>hardware_interface/EffortJointInterface</hardwareInterface>
+    <xacro:macro name="awesome_leg" params="id base_link" >
+        <xacro:unless value="${ base_link=='None' or base_link=='none'}">
+            <!-- only add joint to base if argument is non-empty -->
+            <joint name="hip_pitch${id}" type="revolute">
+                <parent link="${base_link}" />
+                <child link="femur${id}" />
+                <axis xyz="0 1 0"/>
+                <origin xyz="0 ${214.6 * mmTom} 0" />
+                <limit effort="112" lower="-2.4" upper="2.4" velocity="20.0"/>
+            </joint>
+        </xacro:unless>
+        <link name="femur${id}">
+            <inertial>
+                <origin xyz="0.0 0.0 0.0"/>
+                <mass value="3.3712777"/>
+                <inertia ixx="${4.6647423e+04 * kgmm2_2_kgm2}" iyy="${4.3720135e+04 * kgmm2_2_kgm2}" izz="${7.5794813e+04 * kgmm2_2_kgm2}"
+                    ixy="${-1.2697640e+01 * kgmm2_2_kgm2}" ixz="${-3.2745810e+01 * kgmm2_2_kgm2}" iyz="${-6.3299091e+04 * kgmm2_2_kgm2}" />
+            </inertial>
+            <visual>
+                <origin rpy="0.0 0.0 0.0" xyz="0.0 0.0 0.0"/>
+                <geometry>
+                    <mesh filename="package://awesome_leg/description/new_meshes/visual/femur.stl" scale="${dmTom} ${dmTom} ${dmTom}"/>
+                </geometry>
+                <material name="darkblue"/>
+            </visual>
+            <collision>
+                <origin rpy="0.0 0.0 0.0" xyz="0.0 0.0 0.0"/>
+                <geometry>
+                    <mesh filename="package://awesome_leg/description/new_meshes/collision/femur.stl" scale="${dmTom} ${dmTom} ${dmTom}"/>
+                </geometry>
+            </collision>
+        </link>
+        <joint name="knee_pitch${id}" type="revolute">
+            <parent link="femur${id}"/>
+            <child link="shin${id}"/>
+            <origin rpy="0.0 0.0 0.0" xyz="0.0 ${-118.2 * mmTom} ${-300.0 * mmTom}"/>
+            <axis xyz="0 1 0"/>
+            <limit effort="112" lower="-2.4" upper="2.4" velocity="20.0"/>
         </joint>
-        <actuator name="hip_motor">
-            <hardwareInterface>hardware_interface/EffortJointInterface</hardwareInterface>
-            <mechanicalReduction>1</mechanicalReduction>
-        </actuator>
-    </transmission>
-    <transmission name="knee_trans">
-        <type>transmission_interface/SimpleTransmission</type>
-        <joint name="knee_pitch_1">
-            <hardwareInterface>hardware_interface/EffortJointInterface</hardwareInterface>
+        <link name="shin${id}">
+            <inertial>
+                <origin xyz="0.0 0.0 0.0"/>
+                <mass value="1.3106594"/>
+                <inertia ixx="${4.0133965e+04 * kgmm2_2_kgm2}" iyy="${4.0269285e+04 * kgmm2_2_kgm2}" izz="${1.5274496e+03 * kgmm2_2_kgm2}"
+                    ixy="${4.6219082e-02 * kgmm2_2_kgm2}" ixz="${-3.0432320e-01 * kgmm2_2_kgm2}" iyz="${1.3816329e+03 * kgmm2_2_kgm2}" />
+            </inertial>
+            <visual>
+                <origin rpy="0.0 0.0 0.0" xyz="0.0 0.0 0.0"/>
+                <geometry>
+                    <mesh filename="package://awesome_leg/description/new_meshes/visual/shin.stl" scale="${dmTom} ${dmTom} ${dmTom}"/>
+                </geometry>
+                <material name="grey"/>
+            </visual>
+            <collision>
+                <origin rpy="0.0 0.0 0.0" xyz="0.0 0.0 0.0"/>
+                <geometry>
+                    <mesh filename="package://awesome_leg/description/new_meshes/collision/shin.stl" scale="${dmTom} ${dmTom} ${dmTom}"/>
+                </geometry>
+            </collision>
+        </link>
+        <joint name="tip_joint${id}" type="fixed">
+            <parent link="shin${id}"/>
+            <child link="tip${id}"/>
+            <origin xyz="0.0 ${23.3000 * mmTom} ${-451 * mmTom}"/>
         </joint>
-        <actuator name="knee_motor">
-            <hardwareInterface>hardware_interface/EffortJointInterface</hardwareInterface>
-            <mechanicalReduction>1</mechanicalReduction>
-        </actuator>
-    </transmission>
-    <!-- xbot2 joint device driver-->
-    <gazebo>
-        <plugin name='xbot2_gz_joint_server' filename='libxbot2_gz_joint_server.so'>
-            <pid>
-                <gain name="null_mode"  p="0"  d="0"/>
-                <gain name="small_mot"  p="250"  d="5"/>
-                <gain name="medium_mot" p="1000" d="10"/>
-                <gain name="big_mot"    p="3000" d="10"/>
-                <gain name="test_rig2HIP" profile="null_mode"/>
-                <gain name="hip_actuation" profile="medium_mot"/>
-                <gain name="knee_actuation" profile="medium_mot"/>
-            </pid>
-        </plugin>
-    </gazebo>
-    <gazebo>
-        <plugin name="xbot2_ft_driver" filename="libxbot2_gz_ft_server.so"/>
-    </gazebo>
-    <!--Gazebo-specific tags-->
-    <gazebo reference="pelvis">
-    <material>Gazebo/Grey  </material>
-    </gazebo>
-    <gazebo reference="hip1_1">
-        <material>Gazebo/Grey   </material>
-    </gazebo>
-    <gazebo reference="hip2_1">
-        <material>Gazebo/SkyBlue </material>
-    </gazebo>
-    <gazebo reference="knee_1">
-        <material>Gazebo/Grey  </material>
-    </gazebo>
+        <link name="tip${id}"/>
+        <!-- <transmission name="hip_pitch${id}">
+            <type>transmission_interface/SimpleTransmission</type>
+            <joint name="hip_pitch_1">
+                <hardwareInterface>hardware_interface/EffortJointInterface</hardwareInterface>
+            </joint>
+            <actuator name="hip_motor">
+                <hardwareInterface>hardware_interface/EffortJointInterface</hardwareInterface>
+                <mechanicalReduction>1</mechanicalReduction>
+            </actuator>
+        </transmission>
+        <transmission name="knee_trans">
+            <type>transmission_interface/SimpleTransmission</type>
+            <joint name="knee_pitch_1">
+                <hardwareInterface>hardware_interface/EffortJointInterface</hardwareInterface>
+            </joint>
+            <actuator name="knee_motor">
+                <hardwareInterface>hardware_interface/EffortJointInterface</hardwareInterface>
+                <mechanicalReduction>1</mechanicalReduction>
+            </actuator>
+        </transmission> -->
+    </xacro:macro>
 </robot>

File: description/urdf/awesome_leg_standalone.urdf.xacro (robot description, xacro)
@@ -1,11 +1,11 @@
 <?xml version="1.0" encoding="utf-8" ?>
 <!--
-    Leg urdf for use with Cartesio (added world link) and RBDL
+    Leg base URDF (no external links). Variant of the URDF adapted for use with Pinocchio and for performing inertial parameter identification
 -->
 <robot name="awesome_leg" xmlns:xacro="http://www.ros.org/wiki/xacro">
+    <xacro:include filename="$(find awesome_leg)/description/urdf/utils.urdf.xacro" />
     <xacro:include filename="$(find awesome_leg)/description/urdf/utils.urdf.xacro"/>
     <xacro:include filename="$(find awesome_leg)/description/urdf/awesome_leg.xbot.xacro"/>
-    <xacro:include filename="$(find awesome_leg)/description/urdf/awesome_leg.urdf.xacro"/>
-    <link name="world"> </link>
+    <xacro:include filename="$(find awesome_leg)/description/urdf/awesome_leg.urdf.xacro" />
     <xacro:awesome_leg id="1" base_link="none"/>
   </robot>

File: description/urdf/awesome_leg_standalone_calibrated.urdf.xacro (robot description, xacro)
@@ -1,13 +1,16 @@
 <?xml version="1.0" encoding="utf-8" ?>
 <!--
-    Leg base URDF (no external links). Variant of the URDF adapted for use with Pinocchio and for performing inertial parameter identification
+    Leg modified base URDF (basically a simple double pendulum), with calibrated inertial parameters.
+    It is the awesome_leg_standalone.urdf file with modified inertial parameters obtained via an
+    identification procedure.
 -->
 <robot name="awesome_leg" xmlns:xacro="http://www.ros.org/wiki/xacro">
     <xacro:include filename="$(find awesome_leg)/description/urdf/utils.urdf.xacro" />
-    <link name="pelvis"/>
+    <link name="pelvis">
+    </link>
     <joint name="hip_pitch_1" type="revolute">
         <parent link="pelvis"/>
         <child link="shank"/>
-        <origin rpy="-1.57079632679 0 0" xyz="0.0 0.0 0.0"/>
+        <origin rpy="-1.57079632679 0 -1.57079632679" xyz="0.0 0.0 0.0"/>
         <axis xyz="0 0 1"/>
         <limit effort="112" lower="-2.0226" upper="2.02748" velocity="20.0"/>
@@ -15,5 +18,5 @@
     <link name="shank">
         <inertial>
-        <origin xyz="2.57966e-05 0.1810266 0.085669756"/>
+        <origin xyz="2.02539722e-03 2.36232975e-01 8.56697560e-02"/>
         <mass value="2.7264471"/>
         <inertia ixx="0.04851869" ixy="-4.11894e-05" ixz="-1.68778e-05" iyy="0.004242055" iyz="0.0032243188" izz="0.04825583"/>
@@ -33,5 +36,5 @@
         </collision>
     </link>
-     <joint name="knee_pitch_1" type="revolute">
+    <joint name="knee_pitch_1" type="revolute">
         <parent link="shank"/>
         <child link="shin"/>
@@ -42,6 +45,6 @@
     <link name="shin">
         <inertial>
-        <mass value="1.1927236"/>
-        <origin xyz="0.19572282 -0.014549221 -0.020785942"/>
+        <mass value="1.23787877e+00"/>
+        <origin xyz="1.52366156e-01 -3.92736885e-04 -2.00277153e-02"/>
         <inertia ixx="0.0013302597" ixy="0.00060307457" ixz="0.0" iyy="0.035313402" iyz="-1.1029574e-07" izz="0.035530025"/>
         </inertial>

File: description/urdf/awesome_leg_test_rig.urdf.xacro (robot description, xacro)
@@ -1,21 +1,13 @@
 <?xml version="1.0"?>
-<!--
-    Leg complete xacro
--->
 <robot name="awesome_leg" xmlns:xacro="http://www.ros.org/wiki/xacro">
+    <xacro:include filename="$(find awesome_leg)/description/urdf/utils.urdf.xacro"/>
+    <xacro:include filename="$(find awesome_leg)/description/urdf/awesome_leg.xbot.xacro"/>
+    <xacro:include filename="$(find awesome_leg)/description/urdf/awesome_leg.urdf.xacro"/>
     <xacro:arg name="sliding_guide" default="true" />
-    <xacro:arg name="calibrated_urdf" default="true" />
     <xacro:property name="test_rig_base_ext" value="0.1" />
     <xacro:property name="test_rig_height" value="1.0" />
     <xacro:property name="hip_mounting_offset" value="0.08" />
-    <xacro:if value = "$(arg calibrated_urdf)">
-        <xacro:property name="pelvis_mounting_height" value="0.25" />
-    </xacro:if>
-    <xacro:unless value = "$(arg calibrated_urdf)">
-        <xacro:property name="pelvis_mounting_height" value="0.3691" />
-    </xacro:unless>
-    <xacro:property name="payload_mass" value="7.38" />
+    <xacro:property name="pelvis_mounting_height" value="0.0" />
     <link name="world" />
-    <!-- fixing the test rig to the world -->
     <joint name="world_test_rig" type="fixed">
         <parent link="world" />
@@ -38,14 +30,13 @@
         </collision>
         <inertial>
-            <mass value="0.001" />
-            <inertia ixx="0.0001" iyy="0.0001" izz="0.0001" ixy="0.0" ixz="0.0" iyz="0.0" />
+            <mass value="1000.0" />
+            <inertia ixx="0.01" iyy="0.0001" izz="0.0001" ixy="0.0" ixz="0.0" iyz="0.0" />
         </inertial>
     </link>
     <xacro:if value="$(arg sliding_guide)">
-        <!-- Adding a prismatic sliding guide -->
-        <joint name="test_rig2payload" type="prismatic">
+        <joint name="test_rig2base" type="prismatic">
             <parent link="test_rig" />
-            <child link="payload_link" />
-            <origin xyz="${test_rig_base_ext + hip_mounting_offset} 0 ${pelvis_mounting_height}" />
+            <child link="base_link" />
+            <origin xyz="${test_rig_base_ext + hip_mounting_offset} 0 ${pelvis_mounting_height}" rpy="0.0 0.0 ${-PI_2}"/>
             <axis xyz="0 0 1" />
             <dynamics damping="0.0" friction="0.0" />
@@ -54,27 +45,30 @@
     </xacro:if>
     <xacro:unless value="$(arg sliding_guide)">
-        <!-- Adding a prismatic sliding guide -->
-        <joint name="test_rig2payload" type="fixed">
+        <joint name="test_rig2base" type="fixed">
             <parent link="test_rig" />
-            <child link="payload_link" />
-            <origin xyz="${test_rig_base_ext + hip_mounting_offset} 0 ${pelvis_mounting_height}" />
+            <child link="base_link" />
+            <origin xyz="${test_rig_base_ext + hip_mounting_offset} 0 ${pelvis_mounting_height}" rpy="0.0 0.0 ${-PI_2}"/>
         </joint>
     </xacro:unless>
-    <link name="payload_link">
+    <link name="base_link">
+        <visual name="base_link_visual">
+            <origin xyz="0.0 0.0 0.0" rpy="0.0 0.0 0.0"/>
+            <geometry>
+                <mesh filename="package://awesome_leg/description/new_meshes/visual/base.stl" scale="${dmTom} ${dmTom} ${dmTom}"/>
+            </geometry>
+            <material name="black"/>
+        </visual>
+        <collision>
+            <origin xyz="0.0 0.0 0.0" rpy="0.0 0.0 0.0"/>
+            <geometry>
+                <mesh filename="package://awesome_leg/description/new_meshes/collision/base.stl" scale="${dmTom} ${dmTom} ${dmTom}"/>
+            </geometry>
+        </collision>
         <inertial>
-            <mass value="${payload_mass}" />
-            <inertia ixx="0.00001" iyy="0.00001" izz="0.00001" ixy="0.0" ixz="0.0" iyz="0.0" />
+            <mass value="${4.5477704 + payload_mass}" />
+            <inertia ixx="${4.4624842e+04 * kgmm2_2_kgm2}" iyy="${2.6977590e+04 * kgmm2_2_kgm2}" izz="${2.7956754e+04 * kgmm2_2_kgm2}"
+                    ixy="${-1.4644878e+01 * kgmm2_2_kgm2}" ixz="${3.0225947e+01 * kgmm2_2_kgm2}" iyz="${9.6636358e+03 * kgmm2_2_kgm2}" />
         </inertial>
     </link>
-    <joint name="test_rig2shank" type="fixed">
-            <parent link="payload_link" />
-            <child link="pelvis" />
-            <origin xyz="0 0 0" />
-    </joint>
-    <xacro:if value = "$(arg calibrated_urdf)">
-        <xacro:include filename="$(find awesome_leg)/description/urdf/generated/awesome_leg_reduced_calibrated.urdf" />
-    </xacro:if>
-    <xacro:unless value="$(arg calibrated_urdf)">
-        <xacro:include filename="$(find awesome_leg)/description/urdf/awesome_leg.urdf.xacro" />
-    </xacro:unless>
+    <xacro:awesome_leg id="1" base_link="base_link"/>
 </robot>

File: description/urdf/generated/awesome_leg_standalone.urdf (robot description, URDF)
Before this commit: robot awesome_leg, 6 links, 5 joints
Links:
- removed link base_link
- removed link test_rig
- removed link world
Joints:
- removed joint hip_pitch1
- removed joint test_rig2base
- removed joint world_test_rig

File: description/urdf/utils.urdf.xacro (robot description, xacro)
@@ -3,10 +3,14 @@
 <!-- scale -->
 <xacro:property name="mmTom" value="0.001" />
+<xacro:property name="dmTom" value="0.1" />
 <xacro:property name="mm2Tom2" value="${0.001*0.001}" />
 <xacro:property name="tonsToKg" value="1000.0" />
+<xacro:property name="kgmm2_2_kgm2" value="${1e-06}" />
 <xacro:property name="PI" value="3.14159265359" />
 <xacro:property name="PI_2" value="1.57079632679" />
 <xacro:property name="PI_4" value="0.7853981633974483" />
 <xacro:property name="DEG2RAD" value="${PI/180.0}" />
+<xacro:property name="payload_mass" value="0.0" />
+<!-- <xacro:property name="payload_mass" value="7.38" /> -->
 <!-- color -->
 <material name="darkblue">
