Commit message: small aesthetic changes

File: description/urdf/awesome_leg.gazebo.xacro (robot description, xacro)
@@ -1,5 +1,5 @@
 <?xml version="1.0"?>
 <robot xmlns:xacro="http://ros.org/wiki/xacro">
-    <xacro:macro name="awesome_leg" params="id" >
+    <xacro:macro name="awesome_leg_gazebo" params="id" >
     <!--Gazebo-specific tags-->
         <gazebo reference="femur${id}">

File: description/urdf/awesome_leg.urdf.xacro (robot description, xacro)
@@ -3,4 +3,5 @@
     <xacro:include filename="$(find awesome_leg)/description/urdf/awesome_leg.gazebo.xacro" />
     <xacro:macro name="awesome_leg" params="id base_link" >
+        <xacro:awesome_leg_gazebo id="${id}"/>
         <xacro:unless value="${ base_link=='None' or base_link=='none'}">
             <!-- only add joint to base if argument is non-empty -->

File: description/urdf/awesome_leg_test_rig.urdf.xacro (robot description, xacro)
@@ -31,5 +31,5 @@
         <inertial>
             <mass value="1000.0" />
-            <inertia ixx="0.01" iyy="0.0001" izz="0.0001" ixy="0.0" ixz="0.0" iyz="0.0" />
+            <inertia ixx="0.01" iyy="0.01" izz="0.01" ixy="0.0" ixz="0.0" iyz="0.0" />
         </inertial>
     </link>

File: description/urdf/generated/awesome_leg_test_rig.urdf (robot description, URDF)
Before this commit: robot awesome_leg, 6 links, 5 joints
Joints:
- joint test_rig2base: origin xyz=0.18 0 0.0 rpy=0.0 0.0 -1.57079632679 -> xyz=0.18 0 0.25 rpy=0.0 0.0 -1.57079632679

Commit message: some changes

File: description/urdf/awesome_leg.gazebo.xacro (robot description, xacro)
@@ -15,6 +15,6 @@
                     <friction>
                         <ode>
-                            <mu>10</mu>
-                            <mu2>10</mu2>
+                            <mu>20</mu>
+                            <mu2>20</mu2>
                         </ode>
                         <bullet>

File: description/urdf/awesome_leg.xbot.xacro (robot description, xacro)
@@ -18,3 +18,10 @@
         <plugin name="xbot2_ft_driver" filename="libxbot2_gz_ft_server.so"/>
     </gazebo>
+    <gazebo>
+        <plugin name="xbot2_link_state_sensor" filename="libxbot2_gz_link_state_sensor.so">
+            <links>
+                <link name="base_link"/>
+            </links>
+        </plugin>
+    </gazebo>
 </robot>

Commit message: many improvs; first nice jump with lowered impedance
Signed-off-by: andrea patrizi <andrepatrizi1b6e6@gmail.com>

File: description/urdf/awesome_leg.gazebo.xacro (robot description, xacro)
@@ -39,4 +39,28 @@
             </collision>
         </gazebo>
+        <!-- <xacro:if value="${ dump_video_frames== True}">
+            <gazebo reference="camera">
+                <sensor name="my_camera" type="camera">
+                    <camera>
+                        <save enabled="true">
+                            <path "$(find awesome_leg)/description/urdf/utils.urdf.xacro" >
+                        </save>
+                        <horizontal_fov>1</horizontal_fov>
+                        <image>
+                        <width>1920</width>
+                        <height>1080</height>
+                        </image>
+                        <clip>
+                        <near>0.1</near>
+                        <far>100</far>
+                        </clip>
+                        <view_controller>orbit</view_controller>
+                    </camera>
+                    <always_on>1</always_on>
+                    <visualize>false</visualize>
+                    <update_rate>30</update_rate>
+                </sensor>
+            </gazebo>
+        </xacro:if> -->
     </xacro:macro>
 </robot>

File: description/urdf/awesome_leg_test_rig.urdf.xacro (robot description, xacro)
@@ -6,8 +6,25 @@
     <xacro:include filename="$(find awesome_leg)/description/urdf/test_rig.gazebo.xacro"/>
     <xacro:arg name="sliding_guide" default="true" />
+    <xacro:arg name="dump_video_frames" default="false" />
     <xacro:property name="test_rig_base_ext" value="0.1" />
     <xacro:property name="test_rig_height" value="1.0" />
     <xacro:property name="hip_mounting_offset" value="0.08" />
     <xacro:property name="pelvis_mounting_height" value="0.25" />
+    <!-- <xacro:if value="$(arg dump_video_frames)">
+        <joint name="test_rig_2camera_link" type="fixed">
+        <parent link="test_rig" />
+        <child link="camera_link" />
+        <origin xyz="0 ${camera_depth} ${camera_height}" rpy="0 0 0" />
+        </joint>
+        <link name="camera_link">
+            <visual name="visual">
+            <geometry>
+            <box>
+            <size>0.1 0.1 0.1</size>
+            </box>
+            </geometry>
+            </visual>
+        </link>
+    </xacro:if> -->
     <link name="world" />
     <joint name="world_test_rig" type="fixed">

File: description/urdf/generated/awesome_leg.urdf (robot description, URDF)
Before this commit: robot awesome_leg, 6 links, 5 joints
Joints:
- joint knee_pitch1: axis 0 1 0 -> 0 -1 0

File: description/urdf/generated/awesome_leg_standalone.urdf (robot description, URDF)
Before this commit: robot awesome_leg, 3 links, 2 joints
Joints:
- joint knee_pitch1: axis 0 1 0 -> 0 -1 0

File: description/urdf/generated/awesome_leg_xbot.urdf (robot description, URDF)
Before this commit: robot awesome_leg, 5 links, 4 joints
Joints:
- joint knee_pitch1: axis 0 1 0 -> 0 -1 0

File: description/urdf/utils.urdf.xacro (robot description, xacro)
@@ -13,4 +13,6 @@
 <xacro:property name="payload_mass" value="0.0" />
 <!-- <xacro:property name="payload_mass" value="7.38" /> -->
+<xacro:property name="camera_height" value="0.5" />
+<xacro:property name="camera_depth" value="1.0" />
 <!-- color -->
 <material name="darkblue">

Commit message: ft sensor to be added

File: description/urdf/awesome_leg.gazebo.xacro (robot description, xacro)
@@ -1,5 +1,5 @@
 <?xml version="1.0"?>
 <robot xmlns:xacro="http://ros.org/wiki/xacro">
-    <xacro:macro name="awesome_leg_gazebo" params="id" >
+    <xacro:macro name="awesome_leg_gazebo" params="id add_ft_sensor"  >
     <!--Gazebo-specific tags-->
         <gazebo reference="femur${id}">
@@ -63,4 +63,27 @@
             </gazebo>
         </xacro:if> -->
+        <xacro:if value="${ add_ft_sensor == True}">
+            <!-- <link name="ft_sensor${id}">
+                <inertial>
+                    <origin xyz="0.0 0.0 0.0"/>
+                    <mass value=""/>
+                    <inertia ixx="${4.6647423e+04 * kgmm2_2_kgm2}" iyy="${4.3720135e+04 * kgmm2_2_kgm2}" izz="${7.5794813e+04 * kgmm2_2_kgm2}"
+                        ixy="${-1.2697640e+01 * kgmm2_2_kgm2}" ixz="${-3.2745810e+01 * kgmm2_2_kgm2}" iyz="${-6.3299091e+04 * kgmm2_2_kgm2}" />
+                </inertial>
+                <visual>
+                    <origin rpy="0.0 0.0 0.0" xyz="0.0 0.0 0.0"/>
+                    <geometry>
+                        <mesh filename="package://awesome_leg/description/new_meshes/visual/femur.stl" scale="${dmTom} ${dmTom} ${dmTom}"/>
+                    </geometry>
+                    <material name="darkblue"/>
+                </visual>
+                <collision>
+                    <origin rpy="0.0 0.0 0.0" xyz="0.0 0.0 0.0"/>
+                    <geometry>
+                        <mesh filename="package://awesome_leg/description/new_meshes/collision/femur.stl" scale="${dmTom} ${dmTom} ${dmTom}"/>
+                    </geometry>
+                </collision>
+            </link> -->
+        </xacro:if>
     </xacro:macro>
 </robot>

File: description/urdf/awesome_leg.urdf.xacro (robot description, xacro)
@@ -2,6 +2,6 @@
 <robot name="awesome_leg" xmlns:xacro="http://www.ros.org/wiki/xacro">
     <xacro:include filename="$(find awesome_leg)/description/urdf/awesome_leg.gazebo.xacro" />
-    <xacro:macro name="awesome_leg" params="id base_link" >
-        <xacro:awesome_leg_gazebo id="${id}"/>
+    <xacro:macro name="awesome_leg" params="id base_link add_ft_sensor" >
+        <xacro:awesome_leg_gazebo id="${id} ${add_ft_sensor}"/>
         <xacro:unless value="${ base_link=='None' or base_link=='none'}">
             <!-- only add joint to base if argument is non-empty -->

File: description/urdf/awesome_leg_test_rig.urdf.xacro (robot description, xacro)
@@ -6,4 +6,5 @@
     <xacro:include filename="$(find awesome_leg)/description/urdf/test_rig.gazebo.xacro"/>
     <xacro:arg name="sliding_guide" default="true" />
+    <xacro:arg name="add_ft_sensor" default="false" />
     <xacro:arg name="dump_video_frames" default="false" />
     <xacro:property name="test_rig_base_ext" value="0.1" />
@@ -89,4 +90,25 @@
         </inertial>
     </link>
-    <xacro:awesome_leg id="1" base_link="base_link"/>
+    <xacro:awesome_leg id="1" base_link="base_link" add_ft_sensor="$(arg add_ft_sensor)"/>
+    <link name="femur${id}">
+            <inertial>
+                <origin xyz="0.0 0.0 0.0"/>
+                <mass value="3.3712777"/>
+                <inertia ixx="${4.6647423e+04 * kgmm2_2_kgm2}" iyy="${4.3720135e+04 * kgmm2_2_kgm2}" izz="${7.5794813e+04 * kgmm2_2_kgm2}"
+                    ixy="${-1.2697640e+01 * kgmm2_2_kgm2}" ixz="${-3.2745810e+01 * kgmm2_2_kgm2}" iyz="${-6.3299091e+04 * kgmm2_2_kgm2}" />
+            </inertial>
+            <visual>
+                <origin rpy="0.0 0.0 0.0" xyz="0.0 0.0 0.0"/>
+                <geometry>
+                    <mesh filename="package://awesome_leg/description/new_meshes/visual/femur.stl" scale="${dmTom} ${dmTom} ${dmTom}"/>
+                </geometry>
+                <material name="darkblue"/>
+            </visual>
+            <collision>
+                <origin rpy="0.0 0.0 0.0" xyz="0.0 0.0 0.0"/>
+                <geometry>
+                    <mesh filename="package://awesome_leg/description/new_meshes/collision/femur.stl" scale="${dmTom} ${dmTom} ${dmTom}"/>
+                </geometry>
+            </collision>
+    </link>
 </robot>

Commit message: added optional ft sensor and calibrated contact parameters

File: description/urdf/awesome_leg.gazebo.xacro (robot description, xacro)
@@ -11,10 +11,10 @@
         <gazebo reference="shin${id}">
             <collision>
-                <max_contacts> 1 </max_contacts>
+                <max_contacts> 20 </max_contacts>
                 <surface>
                     <friction>
                         <ode>
-                            <mu>20</mu>
-                            <mu2>20</mu2>
+                            <mu>1</mu>
+                            <mu2>1</mu2>
                         </ode>
                         <bullet>
@@ -36,4 +36,34 @@
                         </bullet>
                     </contact> -->
+                </surface>
+            </collision>
+        </gazebo>
+        <gazebo reference="tip${id}">
+            <collision>
+                <max_contacts> 1 </max_contacts>
+                <surface>
+                    <friction>
+                        <ode>
+                            <mu>20</mu>
+                            <mu2>20</mu2>
+                        </ode>
+                        <bullet>
+                            <friction>1.0</friction>
+                            <friction2>1.0</friction2>
+                        </bullet>
+                    </friction>
+                    <contact>
+                        <ode>
+                            <kp>1000000000000</kp>
+                            <kd>1</kd>
+                            <!-- <max_vel>100</max_vel> -->
+                        </ode>
+                        <!-- <bullet>
+                            <soft_cfm>0.007</soft_cfm>
+                            <soft_erp>0.25</soft_erp>
+                            <kp>1000000</kp>
+                            <kd>5</kd>
+                        </bullet> -->
+                    </contact>
                 </surface>
             </collision>
@@ -64,25 +94,16 @@
         </xacro:if> -->
         <xacro:if value="${ add_ft_sensor == True}">
-            <!-- <link name="ft_sensor${id}">
-                <inertial>
-                    <origin xyz="0.0 0.0 0.0"/>
-                    <mass value=""/>
-                    <inertia ixx="${4.6647423e+04 * kgmm2_2_kgm2}" iyy="${4.3720135e+04 * kgmm2_2_kgm2}" izz="${7.5794813e+04 * kgmm2_2_kgm2}"
-                        ixy="${-1.2697640e+01 * kgmm2_2_kgm2}" ixz="${-3.2745810e+01 * kgmm2_2_kgm2}" iyz="${-6.3299091e+04 * kgmm2_2_kgm2}" />
-                </inertial>
-                <visual>
-                    <origin rpy="0.0 0.0 0.0" xyz="0.0 0.0 0.0"/>
-                    <geometry>
-                        <mesh filename="package://awesome_leg/description/new_meshes/visual/femur.stl" scale="${dmTom} ${dmTom} ${dmTom}"/>
-                    </geometry>
-                    <material name="darkblue"/>
-                </visual>
-                <collision>
-                    <origin rpy="0.0 0.0 0.0" xyz="0.0 0.0 0.0"/>
-                    <geometry>
-                        <mesh filename="package://awesome_leg/description/new_meshes/collision/femur.stl" scale="${dmTom} ${dmTom} ${dmTom}"/>
-                    </geometry>
-                </collision>
-            </link> -->
+            <gazebo reference="tip_joint${id}">
+                <sensor type="force_torque" name="tip${id}_fts">
+                    <force_torque>
+                        <frame>sensor</frame>
+                        <measure_direction>child_to_parent</measure_direction>
+                    </force_torque>
+                    <always_on>true</always_on>
+                    <visualize>true</visualize>
+                    <update_rate>1000</update_rate>
+                    <pose>0.0 0.0 0.0 0.0 0.0 0.0</pose> <!-- check! -->
+              </sensor>
+            </gazebo>
         </xacro:if>
     </xacro:macro>

File: description/urdf/awesome_leg.urdf.xacro (robot description, xacro)
@@ -3,5 +3,5 @@
     <xacro:include filename="$(find awesome_leg)/description/urdf/awesome_leg.gazebo.xacro" />
     <xacro:macro name="awesome_leg" params="id base_link add_ft_sensor" >
-        <xacro:awesome_leg_gazebo id="${id} ${add_ft_sensor}"/>
+        <xacro:awesome_leg_gazebo id="${id}" add_ft_sensor="${add_ft_sensor}"/>
         <xacro:unless value="${ base_link=='None' or base_link=='none'}">
             <!-- only add joint to base if argument is non-empty -->
@@ -63,30 +63,36 @@
             </collision>
         </link>
-        <joint name="tip_joint${id}" type="fixed">
-            <parent link="shin${id}"/>
-            <child link="tip${id}"/>
-            <origin xyz="0.0 ${23.3000 * mmTom} ${-451 * mmTom}"/>
-        </joint>
-        <link name="tip${id}"/>
-        <!-- <transmission name="hip_pitch${id}">
-            <type>transmission_interface/SimpleTransmission</type>
-            <joint name="hip_pitch_1">
-                <hardwareInterface>hardware_interface/EffortJointInterface</hardwareInterface>
+        <xacro:unless value="${ add_ft_sensor == True}">
+            <joint name="tip_joint${id}" type="fixed">
+                <parent link="shin${id}"/>
+                <child link="tip${id}"/>
+                <origin xyz="0.0 ${23.3000 * mmTom} ${-451 * mmTom}"/>
             </joint>
-            <actuator name="hip_motor">
-                <hardwareInterface>hardware_interface/EffortJointInterface</hardwareInterface>
-                <mechanicalReduction>1</mechanicalReduction>
-            </actuator>
-        </transmission>
-        <transmission name="knee_trans">
-            <type>transmission_interface/SimpleTransmission</type>
-            <joint name="knee_pitch_1">
-                <hardwareInterface>hardware_interface/EffortJointInterface</hardwareInterface>
+            <link name="tip${id}"/>
+        </xacro:unless>
+        <xacro:if value="${ add_ft_sensor == True}">
+            <joint name="tip_joint${id}" type="revolute">
+                <parent link="shin${id}"/>
+                <child link="tip${id}"/>
+                <origin xyz="0.0 ${23.3000 * mmTom} ${-451 * mmTom + fts_sphere_radius - fts_delta}"/>
+                <limit effort="0" lower="0.0" upper="0.0" velocity="0.0"/>
             </joint>
-            <actuator name="knee_motor">
-                <hardwareInterface>hardware_interface/EffortJointInterface</hardwareInterface>
-                <mechanicalReduction>1</mechanicalReduction>
-            </actuator>
-        </transmission> -->
+            <link name="tip${id}">
+                    <origin xyz="0.0 0.0 0.0"/>
+                    <inertial>
+                        <origin xyz="0.0 0.0 0.0"/>
+                        <mass value="0.01"/>
+                        <inertia ixx="0" iyy="0" izz="0"
+                            ixy="0" ixz="0" iyz="0" />
+                    </inertial>
+                    <collision>
+                        <origin rpy="0.0 0.0 0.0" xyz="0.0 0.0 0.0"/>
+                        <geometry>
+                            <sphere radius="${fts_sphere_radius}"/>
+                        </geometry>
+                        <max_contacts> 20 </max_contacts>
+                    </collision>
+            </link>
+        </xacro:if>
     </xacro:macro>
 </robot>

File: description/urdf/awesome_leg_standalone.urdf.xacro (robot description, xacro)
@@ -8,4 +8,4 @@
     <xacro:include filename="$(find awesome_leg)/description/urdf/awesome_leg.xbot.xacro"/>
     <xacro:include filename="$(find awesome_leg)/description/urdf/awesome_leg.urdf.xacro" />
-    <xacro:awesome_leg id="1" base_link="none"/>
+    <xacro:awesome_leg id="1" base_link="none" add_ft_sensor= "false"/>
   </robot>

File: description/urdf/awesome_leg_test_rig.urdf.xacro (robot description, xacro)
@@ -6,5 +6,5 @@
     <xacro:include filename="$(find awesome_leg)/description/urdf/test_rig.gazebo.xacro"/>
     <xacro:arg name="sliding_guide" default="true" />
-    <xacro:arg name="add_ft_sensor" default="false" />
+    <xacro:arg name="add_ft_sensor" default="true" />
     <xacro:arg name="dump_video_frames" default="false" />
     <xacro:property name="test_rig_base_ext" value="0.1" />
@@ -91,24 +91,3 @@
     </link>
     <xacro:awesome_leg id="1" base_link="base_link" add_ft_sensor="$(arg add_ft_sensor)"/>
-    <link name="femur${id}">
-            <inertial>
-                <origin xyz="0.0 0.0 0.0"/>
-                <mass value="3.3712777"/>
-                <inertia ixx="${4.6647423e+04 * kgmm2_2_kgm2}" iyy="${4.3720135e+04 * kgmm2_2_kgm2}" izz="${7.5794813e+04 * kgmm2_2_kgm2}"
-                    ixy="${-1.2697640e+01 * kgmm2_2_kgm2}" ixz="${-3.2745810e+01 * kgmm2_2_kgm2}" iyz="${-6.3299091e+04 * kgmm2_2_kgm2}" />
-            </inertial>
-            <visual>
-                <origin rpy="0.0 0.0 0.0" xyz="0.0 0.0 0.0"/>
-                <geometry>
-                    <mesh filename="package://awesome_leg/description/new_meshes/visual/femur.stl" scale="${dmTom} ${dmTom} ${dmTom}"/>
-                </geometry>
-                <material name="darkblue"/>
-            </visual>
-            <collision>
-                <origin rpy="0.0 0.0 0.0" xyz="0.0 0.0 0.0"/>
-                <geometry>
-                    <mesh filename="package://awesome_leg/description/new_meshes/collision/femur.stl" scale="${dmTom} ${dmTom} ${dmTom}"/>
-                </geometry>
-            </collision>
-    </link>
 </robot>

File: description/urdf/awesome_leg_xbot.urdf.xacro (robot description, xacro)
@@ -15,4 +15,4 @@
     </joint>
     <link name="base_link"> </link>
-    <xacro:awesome_leg id="1" base_link="base_link"/>
+    <xacro:awesome_leg id="1" base_link="base_link" add_ft_sensor= "false"/>
   </robot>

File: description/urdf/generated/awesome_leg.urdf (robot description, URDF)
Before this commit: robot awesome_leg, 6 links, 5 joints
Links:
- link tip1: mass None -> 0.1; geometry collision sphere radius=0.045
Joints:
- joint tip_joint1: limit (none) -> lower=0.0 upper=0.0 effort=0 velocity=0.0; origin xyz=0.0 0.0233 -0.451 -> xyz=0.0 0.0233 -0.40900000000000003; type fixed -> revolute

File: description/urdf/utils.urdf.xacro (robot description, xacro)
@@ -15,4 +15,6 @@
 <xacro:property name="camera_height" value="0.5" />
 <xacro:property name="camera_depth" value="1.0" />
+<xacro:property name="fts_sphere_radius" value="0.045" />
+<xacro:property name="fts_delta" value="0.003" />
 <!-- color -->
 <material name="darkblue">

Commit message: decently working ground truth force torque sensor

File: description/urdf/awesome_leg.gazebo.xacro (robot description, xacro)
@@ -94,5 +94,13 @@
         </xacro:if> -->
         <xacro:if value="${ add_ft_sensor == True}">
+            <gazebo>
+                <plugin name="ft_sensor" filename="libgazebo_ros_ft_sensor.so">
+                    <updateRate>200.0</updateRate>
+                    <topicName>awesome_leg/ft_sensor_tip</topicName>
+                    <jointName>tip_joint${id}</jointName>
+                </plugin>
+            </gazebo>
             <gazebo reference="tip_joint${id}">
+                <provideFeedback>true</provideFeedback>
                 <sensor type="force_torque" name="tip${id}_fts">
                     <force_torque>
@@ -102,6 +110,6 @@
                     <always_on>true</always_on>
                     <visualize>true</visualize>
-                    <update_rate>1000</update_rate>
-                    <pose>0.0 0.0 0.0 0.0 0.0 0.0</pose> <!-- check! -->
+                    <update_rate>200</update_rate>
+                    <pose>0.0 0.0 0.0 0.0 0.0 0.0</pose>
               </sensor>
             </gazebo>

File: description/urdf/awesome_leg.urdf.xacro (robot description, xacro)
@@ -72,9 +72,10 @@
         </xacro:unless>
         <xacro:if value="${ add_ft_sensor == True}">
-            <joint name="tip_joint${id}" type="revolute">
+            <joint name="tip_joint${id}" type="prismatic">
                 <parent link="shin${id}"/>
                 <child link="tip${id}"/>
                 <origin xyz="0.0 ${23.3000 * mmTom} ${-451 * mmTom + fts_sphere_radius - fts_delta}"/>
                 <limit effort="0" lower="0.0" upper="0.0" velocity="0.0"/>
+                <axis  xyz="0 0 1"/>
             </joint>
             <link name="tip${id}">
@@ -82,5 +83,5 @@
                     <inertial>
                         <origin xyz="0.0 0.0 0.0"/>
-                        <mass value="0.01"/>
+                        <mass value="0.005"/> <!-- fake inertial value, otherwise Gazebo throws errors  -->
                         <inertia ixx="0" iyy="0" izz="0"
                             ixy="0" ixz="0" iyz="0" />

File: description/urdf/utils.urdf.xacro (robot description, xacro)
@@ -16,5 +16,5 @@
 <xacro:property name="camera_depth" value="1.0" />
 <xacro:property name="fts_sphere_radius" value="0.045" />
-<xacro:property name="fts_delta" value="0.003" />
+<xacro:property name="fts_delta" value="0.005" />
 <!-- color -->
 <material name="darkblue">
