Commit message: decent contact parameters for gazebo

File: description/urdf/awesome_leg.gazebo.xacro (robot description, xacro)
@@ -45,6 +45,6 @@
                     <friction>
                         <ode>
-                            <mu>20</mu>
-                            <mu2>20</mu2>
+                            <mu>1</mu>
+                            <mu2>1</mu2>
                         </ode>
                         <bullet>

File: description/urdf/awesome_leg.urdf.xacro (robot description, xacro)
@@ -83,5 +83,5 @@
                     <inertial>
                         <origin xyz="0.0 0.0 0.0"/>
-                        <mass value="0.005"/> <!-- fake inertial value, otherwise Gazebo throws errors  -->
+                        <mass value="${aux_mass_tip}"/> <!-- fake inertial value, otherwise Gazebo throws errors  -->
                         <inertia ixx="0" iyy="0" izz="0"
                             ixy="0" ixz="0" iyz="0" />

File: description/urdf/utils.urdf.xacro (robot description, xacro)
@@ -17,4 +17,5 @@
 <xacro:property name="fts_sphere_radius" value="0.045" />
 <xacro:property name="fts_delta" value="0.005" />
+<xacro:property name="aux_mass_tip" value="0.005" />
 <!-- color -->
 <material name="darkblue">

Commit message: added estimate of static friction on the sliding guide

File: description/urdf/awesome_leg.gazebo.xacro (robot description, xacro)
@@ -98,8 +98,8 @@
                     <updateRate>200.0</updateRate>
                     <topicName>awesome_leg/ft_sensor_tip</topicName>
-                    <jointName>tip_joint${id}</jointName>
+                    <jointName>tip_joint_${id}</jointName>
                 </plugin>
             </gazebo>
-            <gazebo reference="tip_joint${id}">
+            <gazebo reference="tip_joint_${id}">
                 <provideFeedback>true</provideFeedback>
                 <sensor type="force_torque" name="tip${id}_fts">

File: description/urdf/awesome_leg_test_rig.urdf.xacro (robot description, xacro)
@@ -59,5 +59,5 @@
             <origin xyz="${test_rig_base_ext + hip_mounting_offset} 0 ${pelvis_mounting_height}" rpy="0.0 0.0 ${-PI_2}"/>
             <axis xyz="0 0 1" />
-            <dynamics damping="0.0" friction="0.0" />
+            <dynamics damping="${sliding_guide_dyn_friction}" friction="${sliding_guide_static_friction}" />
             <limit lower="-10" upper="10.0" effort="500" velocity="50.0" />
         </joint>

File: description/urdf/generated/awesome_leg.urdf (robot description, URDF)
Before this commit: robot awesome_leg, 6 links, 5 joints
Links:
- link base_link: mass 4.5477704 -> 6.5477704

File: description/urdf/utils.urdf.xacro (robot description, xacro)
@@ -11,4 +11,6 @@
 <xacro:property name="PI_4" value="0.7853981633974483" />
 <xacro:property name="DEG2RAD" value="${PI/180.0}" />
+<xacro:property name="sliding_guide_static_friction" value="0.0" />
+<xacro:property name="sliding_guide_dyn_friction" value="50.0" />
 <xacro:property name="base_link_mass_compensation" value="2.0" />
 <xacro:property name="payload_mass" value="${0.0 + base_link_mass_compensation}" />

Commit message: modified contact description

File: description/urdf/awesome_leg.gazebo.xacro (robot description, xacro)
@@ -94,7 +94,11 @@
         </xacro:if> -->
         <xacro:if value="${ add_ft_sensor == True}">
+            <!-- from the Gazebo API: returns "the wrench applied by the child
+            Link on the Joint specified in the child Link frame.
+            Note that this sign convention is opposite of the reaction forces
+            of the Joint on the Links" -->
             <gazebo>
                 <plugin name="ft_sensor" filename="libgazebo_ros_ft_sensor.so">
-                    <updateRate>200.0</updateRate>
+                    <updateRate>0.0</updateRate> <!-- 0.0 is as fast as possible -->
                     <topicName>awesome_leg/ft_sensor_tip</topicName>
                     <jointName>tip_joint_${id}</jointName>
@@ -110,5 +114,5 @@
                     <always_on>true</always_on>
                     <visualize>true</visualize>
-                    <update_rate>200</update_rate>
+                    <update_rate>0.0</update_rate>
                     <pose>0.0 0.0 0.0 0.0 0.0 0.0</pose>
               </sensor>

File: description/urdf/awesome_leg.urdf.xacro (robot description, xacro)
@@ -56,10 +56,12 @@
                 <material name="grey"/>
             </visual>
-            <collision>
-                <origin rpy="0.0 0.0 0.0" xyz="0.0 0.0 0.0"/>
-                <geometry>
-                    <mesh filename="package://awesome_leg/description/new_meshes/collision/shin.stl" scale="${dmTom} ${dmTom} ${dmTom}"/>
-                </geometry>
-            </collision>
+            <xacro:unless value="${ add_ft_sensor == True}">
+                <collision>
+                    <origin rpy="0.0 0.0 0.0" xyz="0.0 0.0 0.0"/>
+                    <geometry>
+                        <mesh filename="package://awesome_leg/description/new_meshes/collision/shin.stl" scale="${dmTom} ${dmTom} ${dmTom}"/>
+                    </geometry>
+                </collision>
+            </xacro:unless>
         </link>
         <xacro:unless value="${ add_ft_sensor == True}">
@@ -75,5 +77,5 @@
                 <parent link="shin${id}"/>
                 <child link="tip${id}"/>
-                <origin xyz="0.0 ${23.3000 * mmTom} ${-451 * mmTom + fts_sphere_radius - fts_delta}"/>
+                <origin xyz="0.0 ${23.3000 * mmTom} ${-451 * mmTom}"/>
                 <limit effort="0" lower="0.0" upper="0.0" velocity="0.0"/>
                 <axis  xyz="0 0 1"/>
@@ -88,5 +90,5 @@
                     </inertial>
                     <collision>
-                        <origin rpy="0.0 0.0 0.0" xyz="0.0 0.0 0.0"/>
+                        <origin rpy="0.0 0.0 0.0" xyz="0.0 0.0 ${fts_sphere_radius - fts_delta}"/>
                         <geometry>
                             <sphere radius="${fts_sphere_radius}"/>

File: description/urdf/utils.urdf.xacro (robot description, xacro)
@@ -19,6 +19,6 @@
 <xacro:property name="camera_height" value="0.5" />
 <xacro:property name="camera_depth" value="1.0" />
-<xacro:property name="fts_sphere_radius" value="0.045" />
-<xacro:property name="fts_delta" value="0.005" />
+<xacro:property name="fts_sphere_radius" value="0.001" />
+<xacro:property name="fts_delta" value="0.000" />
 <xacro:property name="aux_mass_tip" value="0.005" />
 <!-- color -->
