Commit message: small changes

File: description/urdf/awesome_leg.urdf.xacro (robot description, xacro)
@@ -1,33 +1,58 @@
 <?xml version="1.0" encoding="utf-8" ?>
-<!--
-    Leg modified base URDF (basically a simple double pendulum), with calibrated inertial parameters.
-    It is the awesome_leg_reduced.urdf file with modified inertial parameters obtained via an
-    identification procedure.
--->
 <robot name="awesome_leg" xmlns:xacro="http://www.ros.org/wiki/xacro">
-    <material name="sky_blue">
-        <color rgba="0.13 0.44 0.70 1"/>
-    </material>
-    <material name="grey">
-        <color rgba=" 0.6 0.6 0.6 1"/>
-    </material>
-    <material name="black">
-        <color rgba="0.4 0.4 0.4 1"/>
-    </material>
-    <material name="brown">
-        <color rgba="0.59 0.29 0.0 1"/>
-    </material>
-    <link name="pelvis"/>
+    <xacro:include filename="$(find awesome_leg)/urdf/utils.urdf.xacro" />
+    <link name="pelvis">
+        <inertial>
+        <mass value="1.0"/> <!-- here an additional mass contribution can be added to mimic a weight can be added (standard link mass = 1 Kg) -->
+        <inertia ixx="0.00208333333333" ixy="0.0" ixz="0.0" iyy="0.00208333333333" iyz="0.0" izz="0.0025"/>
+        </inertial>
+        <visual>
+        <geometry>
+            <cylinder length="0.1" radius="0.1"/>
+        </geometry>
+        </visual>
+        <visual>
+        <geometry>
+            <cylinder length="0.1" radius="0.1"/>
+        </geometry>
+        </visual>
+    </link>
+    <joint name="hip_yaw_1" type="fixed">
+        <parent link="pelvis"/>
+        <child link="hip1_1"/>
+        <origin rpy="3.14159265359 0.0 0.0" xyz="0.0 -0.0 -0.0566"/>
+    </joint>
+    <link name="hip1_1">
+        <inertial>
+        <origin xyz="0.010214199 0.0 0.038090987"/>
+        <mass value="1.9194403"/>
+        <inertia ixx="0.0047439572" ixy="-0.0" ixz="-0.0003784138" iyy="0.0040551878" iyz="-0.0" izz="0.0034146219"/>
+        </inertial>
+        <visual>
+        <origin rpy="0.0 0.0 2.03221245002" xyz="0.0 0.0 0.0"/>
+        <geometry>
+            <mesh filename="package://awesome_leg/description/meshes/visual/hip-yaw.stl" scale="0.001 0.001 0.001"/>
+        </geometry>
+        <material name="grey"/>
+        </visual>
+        <collision>
+        <origin rpy="0.0 0.0 2.03221245002" xyz="0.0 0.0 0.0"/>
+        <geometry>
+            <mesh filename="package://awesome_leg/description/meshes/collision/hip-yaw.stl" scale="0.001 0.001 0.001"/>
+        </geometry>
+        </collision>
+    </link>
     <joint name="hip_pitch_1" type="revolute">
-        <parent link="pelvis"/>
-        <child link="shank"/>
-        <origin rpy="-1.57079632679 0 -1.57079632679" xyz="0.0 0.0 0.0"/>
+        <parent link="hip1_1"/>
+        <child link="hip2_1"/>
+        <origin rpy="1.57079632679 0.0 1.5707963268" xyz="0.0 0.0 0.0625"/>
         <axis xyz="0 0 1"/>
         <limit effort="112" lower="-2.0226" upper="2.02748" velocity="20.0"/>
     </joint>
-    <link name="shank">
+    <link name="hip2_1"> <!-- #### -->
         <inertial>
-        <origin xyz="2.02539722e-03 2.36232975e-01 8.56697560e-02"/>
+        <origin xyz="2.57966e-05 0.1810266 0.085669756"/>
         <mass value="2.7264471"/>
+        <!-- org: 4.5 -->
         <inertia ixx="0.04851869" ixy="-4.11894e-05" ixz="-1.68778e-05" iyy="0.004242055" iyz="0.0032243188" izz="0.04825583"/>
         </inertial>
@@ -47,14 +72,14 @@
     </link>
     <joint name="knee_pitch_1" type="revolute">
-        <parent link="shank"/>
-        <child link="shin"/>
+        <parent link="hip2_1"/>
+        <child link="knee_1"/>
         <origin rpy="3.14159265359 0.0 1.57079632679" xyz="0.0 0.3 -0.0036"/>
         <axis xyz="0 0 1"/>grey
         <limit effort="112" lower="-2.0226" upper="2.02748" velocity="20.0"/>
     </joint>
-    <link name="shin">
+    <link name="knee_1"> <!-- #### -->
         <inertial>
-        <mass value="1.23787877e+00"/>
-        <origin xyz="1.52366156e-01 -3.92736885e-04 -2.00277153e-02"/>
+        <mass value="1.1927236"/>
+        <origin rpy="0.0 0.0 0.0" xyz="0.19572282 -0.014549221 -0.020785942"/>
         <inertia ixx="0.0013302597" ixy="0.00060307457" ixz="0.0" iyy="0.035313402" iyz="-1.1029574e-07" izz="0.035530025"/>
         </inertial>
@@ -74,10 +99,9 @@
     </link>
     <joint name="tip_joint" type="fixed">
-        <parent link="shin"/>
+        <parent link="knee_1"/>
         <child link="tip"/>
         <origin xyz="0.45 0.0 -0.02"/>
     </joint>
-    <link name="tip">
-    </link>
+    <link name="tip"/> <!-- just for reference-->
     <transmission name="hip_trans">
         <type>transmission_interface/SimpleTransmission</type>

File: description/urdf/awesome_leg_reduced.urdf (robot description, URDF)
Before this commit: robot awesome_leg, 4 links, 3 joints
Links:
- removed link world
- added link pelvis
Joints:
- joint hip_pitch_1: parent world -> pelvis

File: description/urdf/awesome_leg_test_rig.urdf.xacro (robot description, xacro)
@@ -5,9 +5,15 @@
 <robot name="awesome_leg" xmlns:xacro="http://www.ros.org/wiki/xacro">
     <xacro:arg name="sliding_guide" default="true" />
-    <xacro:property name="test_righ_base_ext" value="0.1" />
-    <xacro:property name="test_righ_height" value="1.0" />
+    <xacro:arg name="calibrated_urdf" default="true" />
+    <xacro:property name="test_rig_base_ext" value="0.1" />
+    <xacro:property name="test_rig_height" value="1.0" />
     <xacro:property name="hip_mounting_offset" value="0.08" />
-    <xacro:property name="pelvis_mounting_height" value="0.3691" />
-    <xacro:property name="payload_mass" value="4.0" />
+    <xacro:if value = "$(arg calibrated_urdf)">
+        <xacro:property name="pelvis_mounting_height" value="0.25" />
+    </xacro:if>
+    <xacro:unless value = "$(arg calibrated_urdf)">
+        <xacro:property name="pelvis_mounting_height" value="0.3691" />
+    </xacro:unless>
+    <xacro:property name="payload_mass" value="10.0" />
     <link name="world" />
     <!-- fixing the test rig to the world -->
@@ -15,5 +21,5 @@
         <parent link="world" />
         <child link="test_rig" />
-        <origin xyz="0 0 ${test_righ_height / 2}" />
+        <origin xyz="0 0 ${test_rig_height / 2}" />
     </joint>
     <link name="test_rig">
@@ -21,5 +27,5 @@
             <origin rpy="0 0 0" xyz="0 0 0" />
             <geometry>
-                <box size="${test_righ_base_ext} ${test_righ_base_ext} ${test_righ_height}" />
+                <box size="${test_rig_base_ext} ${test_rig_base_ext} ${test_rig_height}" />
             </geometry>
             <material name="brown"/>
@@ -28,5 +34,5 @@
             <origin rpy="0 0 0" xyz="0 0 0" />
             <geometry>
-                <box size="${test_righ_base_ext} ${test_righ_base_ext} ${test_righ_height}" />
+                <box size="${test_rig_base_ext} ${test_rig_base_ext} ${test_rig_height}" />
             </geometry>
         </collision>
@@ -41,5 +47,5 @@
             <parent link="test_rig" />
             <child link="payload_link" />
-            <origin xyz="${test_righ_base_ext + hip_mounting_offset} 0 ${pelvis_mounting_height}" />
+            <origin xyz="${test_rig_base_ext + hip_mounting_offset} 0 ${pelvis_mounting_height}" />
             <axis xyz="0 0 1" />
             <dynamics damping="0.0" friction="0.0" />
@@ -52,5 +58,5 @@
             <parent link="test_rig" />
             <child link="payload_link" />
-            <origin xyz="${test_righ_base_ext + hip_mounting_offset} 0 ${pelvis_mounting_height}" />
+            <origin xyz="${test_rig_base_ext + hip_mounting_offset} 0 ${pelvis_mounting_height}" />
         </joint>
     </xacro:unless>
@@ -61,9 +67,14 @@
         </inertial>
     </link>
-    <joint name="test_rig2pelvis" type="fixed">
-        <parent link="payload_link" />
-        <child link="pelvis" />
-        <origin xyz="0 0 0" />
-    </joint>
-    <xacro:include filename="$(find awesome_leg)/description/urdf/awesome_leg.urdf" />
+    <joint name="test_rig2shank" type="fixed">
+            <parent link="payload_link" />
+            <child link="pelvis" />
+            <origin xyz="0 0 0" />
+        </joint>
+    <xacro:if value = "$(arg calibrated_urdf)">
+        <xacro:include filename="$(find awesome_leg)/description/urdf/awesome_leg_reduced_calibrated.urdf" />
+    </xacro:if>
+    <xacro:unless value="$(arg calibrated_urdf)">
+        <xacro:include filename="$(find awesome_leg)/description/urdf/awesome_leg.urdf" />
+    </xacro:unless>
 </robot>

File: description/urdf/generated/awesome_leg_test_rig.urdf (robot description, URDF)
Before this commit: robot awesome_leg, 8 links, 7 joints
Links:
- removed link hip1_1
- removed link hip2_1
- removed link knee_1
- added link shank, mass 2.7264471; collision mesh filename=package://awesome_leg/description/meshes/collision/hip-pitc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 scale=0.001 0.001 0.001; visual mesh filename=package://awesome_leg/description/meshes/visual/hip-pitch.s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 scale=0.001 0.001 0.001
- added link shin, mass 1.23787877e+00; collision mesh filename=package://awesome_leg/description/meshes/collision/front_ri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 scale=0.001 0.001 0.001; visual mesh filename=package://awesome_leg/description/meshes/visual/front_right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 scale=0.001 0.001 0.001
- link payload_link: mass 4.0 -> 10.0
- link pelvis: mass 1.0 -> None; geometry 
Joints:
- removed joint hip_yaw_1
- removed joint test_rig2pelvis
- added joint test_rig2shank: type fixed, parent payload_link, child pelvis, origin xyz=0 0 0
- joint hip_pitch_1: child hip2_1 -> shank; origin xyz=0.0 0.0 0.0625 rpy=1.57079632679 0.0 1.5707963268 -> xyz=0.0 0.0 0.0 rpy=-1.57079632679 0 -1.57079632679; parent hip1_1 -> pelvis
- joint knee_pitch_1: child knee_1 -> shin; parent hip2_1 -> shank
- joint test_rig2payload: origin xyz=0.18 0 0.3691 -> xyz=0.18 0 0.25
- joint tip_joint: parent knee_1 -> shin

Commit message: description files improvement

File: description/urdf/awesome_leg.urdf.xacro (robot description, xacro)
@@ -1,5 +1,5 @@
 <?xml version="1.0" encoding="utf-8" ?>
 <robot name="awesome_leg" xmlns:xacro="http://www.ros.org/wiki/xacro">
-    <xacro:include filename="$(find awesome_leg)/urdf/utils.urdf.xacro" />
+    <xacro:include filename="$(find awesome_leg)/description/urdf/utils.urdf.xacro" />
     <link name="pelvis">
         <inertial>

File: description/urdf/awesome_leg_cartesio.urdf.xacro (robot description, xacro)
@@ -10,4 +10,4 @@
         <child link="pelvis"/>
     </joint>
-    <xacro:include filename="$(find awesome_leg)/description/urdf/awesome_leg.urdf" />
+    <xacro:include filename="$(find awesome_leg)/description/urdf/awesome_leg.urdf.xacro" />
   </robot>

File: description/urdf/awesome_leg_test_rig.urdf.xacro (robot description, xacro)
@@ -71,10 +71,10 @@
             <child link="pelvis" />
             <origin xyz="0 0 0" />
-        </joint>
+    </joint>
     <xacro:if value = "$(arg calibrated_urdf)">
         <xacro:include filename="$(find awesome_leg)/description/urdf/awesome_leg_reduced_calibrated.urdf" />
     </xacro:if>
     <xacro:unless value="$(arg calibrated_urdf)">
-        <xacro:include filename="$(find awesome_leg)/description/urdf/awesome_leg.urdf" />
+        <xacro:include filename="$(find awesome_leg)/description/urdf/generated/awesome_leg.urdf.xacro" />
     </xacro:unless>
 </robot>

Commit message: updated joint limits

File: description/urdf/awesome_leg.urdf.xacro (robot description, xacro)
@@ -48,5 +48,5 @@
         <origin rpy="1.57079632679 0.0 1.5707963268" xyz="0.0 0.0 0.0625"/>
         <axis xyz="0 0 1"/>
-        <limit effort="112" lower="-2.0226" upper="2.02748" velocity="20.0"/>
+        <limit effort="112" lower="-2.4" upper="2.4" velocity="20.0"/>
     </joint>
     <link name="hip2_1"> <!-- #### -->
@@ -76,5 +76,5 @@
         <origin rpy="3.14159265359 0.0 1.57079632679" xyz="0.0 0.3 -0.0036"/>
         <axis xyz="0 0 1"/>grey
-        <limit effort="112" lower="-2.0226" upper="2.02748" velocity="20.0"/>
+        <limit effort="112" lower="-2.4" upper="2.4" velocity="20.0"/>
     </joint>
     <link name="knee_1"> <!-- #### -->

File: description/urdf/generated/awesome_leg_cartesio.urdf (robot description, URDF)
Before this commit: robot awesome_leg, 6 links, 5 joints
Joints:
- joint hip_pitch_1: limit lower=-2.0226 upper=2.02748 effort=112 velocity=20.0 -> lower=-2.4 upper=2.4 effort=112 velocity=20.0
- joint knee_pitch_1: limit lower=-2.0226 upper=2.02748 effort=112 velocity=20.0 -> lower=-2.4 upper=2.4 effort=112 velocity=20.0

File: description/urdf/generated/awesome_leg_reduced_calibrated.urdf.xacro (robot description, xacro)
@@ -1,7 +1,12 @@
 <?xml version="1.0" ?>
 <!-- =================================================================================== -->
-<!-- |    This document was autogenerated by xacro from awesome_leg.urdf.xacro         | -->
+<!-- |    This document was autogenerated by xacro from awesome_leg_reduced_calibrated.urdf.xacro | -->
 <!-- |    EDITING THIS FILE BY HAND IS NOT RECOMMENDED                                 | -->
 <!-- =================================================================================== -->
+<!--
+    Leg modified base URDF (basically a simple double pendulum), with calibrated inertial parameters.
+    It is the awesome_leg_reduced.urdf file with modified inertial parameters obtained via an
+    identification procedure.
+-->
 <robot name="awesome_leg">
   <!-- color -->
@@ -25,58 +30,16 @@
   </material>
   <link name="pelvis">
+    </link>
+  <joint name="hip_pitch_1" type="revolute">
+    <parent link="pelvis"/>
+    <child link="shank"/>
+    <origin rpy="-1.57079632679 0 -1.57079632679" xyz="0.0 0.0 0.0"/>
+    <axis xyz="0 0 1"/>
+    <limit effort="112" lower="-2.0226" upper="2.02748" velocity="20.0"/>
+  </joint>
+  <link name="shank">
     <inertial>
-      <mass value="1.0"/>
-      <!-- here an additional mass contribution can be added to mimic a weight can be added (standard link mass = 1 Kg) -->
-      <inertia ixx="0.00208333333333" ixy="0.0" ixz="0.0" iyy="0.00208333333333" iyz="0.0" izz="0.0025"/>
-    </inertial>
-    <visual>
-      <geometry>
-        <cylinder length="0.1" radius="0.1"/>
-      </geometry>
-    </visual>
-    <visual>
-      <geometry>
-        <cylinder length="0.1" radius="0.1"/>
-      </geometry>
-    </visual>
-  </link>
-  <joint name="hip_yaw_1" type="fixed">
-    <parent link="pelvis"/>
-    <child link="hip1_1"/>
-    <origin rpy="3.14159265359 0.0 0.0" xyz="0.0 -0.0 -0.0566"/>
-  </joint>
-  <link name="hip1_1">
-    <inertial>
-      <origin xyz="0.010214199 0.0 0.038090987"/>
-      <mass value="1.9194403"/>
-      <inertia ixx="0.0047439572" ixy="-0.0" ixz="-0.0003784138" iyy="0.0040551878" iyz="-0.0" izz="0.0034146219"/>
-    </inertial>
-    <visual>
-      <origin rpy="0.0 0.0 2.03221245002" xyz="0.0 0.0 0.0"/>
-      <geometry>
-        <mesh filename="package://awesome_leg/description/meshes/visual/hip-yaw.stl" scale="0.001 0.001 0.001"/>
-      </geometry>
-      <material name="grey"/>
-    </visual>
-    <collision>
-      <origin rpy="0.0 0.0 2.03221245002" xyz="0.0 0.0 0.0"/>
-      <geometry>
-        <mesh filename="package://awesome_leg/description/meshes/collision/hip-yaw.stl" scale="0.001 0.001 0.001"/>
-      </geometry>
-    </collision>
-  </link>
-  <joint name="hip_pitch_1" type="revolute">
-    <parent link="hip1_1"/>
-    <child link="hip2_1"/>
-    <origin rpy="1.57079632679 0.0 1.5707963268" xyz="0.0 0.0 0.0625"/>
-    <axis xyz="0 0 1"/>
-    <limit effort="112" lower="-2.4" upper="2.4" velocity="20.0"/>
-  </joint>
-  <link name="hip2_1">
-    <!-- #### -->
-    <inertial>
-      <origin xyz="2.57966e-05 0.1810266 0.085669756"/>
+      <origin xyz="2.02539722e-03 2.36232975e-01 8.56697560e-02"/>
       <mass value="2.7264471"/>
-      <!-- org: 4.5 -->
       <inertia ixx="0.04851869" ixy="-4.11894e-05" ixz="-1.68778e-05" iyy="0.004242055" iyz="0.0032243188" izz="0.04825583"/>
     </inertial>
@@ -96,16 +59,15 @@
   </link>
   <joint name="knee_pitch_1" type="revolute">
-    <parent link="hip2_1"/>
-    <child link="knee_1"/>
+    <parent link="shank"/>
+    <child link="shin"/>
     <origin rpy="3.14159265359 0.0 1.57079632679" xyz="0.0 0.3 -0.0036"/>
     <axis xyz="0 0 1"/>
     grey
-    <limit effort="112" lower="-2.4" upper="2.4" velocity="20.0"/>
+    <limit effort="112" lower="-2.0226" upper="2.02748" velocity="20.0"/>
   </joint>
-  <link name="knee_1">
-    <!-- #### -->
+  <link name="shin">
     <inertial>
-      <mass value="1.1927236"/>
-      <origin rpy="0.0 0.0 0.0" xyz="0.19572282 -0.014549221 -0.020785942"/>
+      <mass value="1.23787877e+00"/>
+      <origin xyz="1.52366156e-01 -3.92736885e-04 -2.00277153e-02"/>
       <inertia ixx="0.0013302597" ixy="0.00060307457" ixz="0.0" iyy="0.035313402" iyz="-1.1029574e-07" izz="0.035530025"/>
     </inertial>
@@ -125,10 +87,10 @@
   </link>
   <joint name="tip_joint" type="fixed">
-    <parent link="knee_1"/>
+    <parent link="shin"/>
     <child link="tip"/>
     <origin xyz="0.45 0.0 -0.02"/>
   </joint>
-  <link name="tip"/>
-  <!-- just for reference-->
+  <link name="tip">
+    </link>
   <transmission name="hip_trans">
     <type>transmission_interface/SimpleTransmission</type>

File: description/urdf/generated/awesome_leg_test_rig.urdf (robot description, URDF)
Before this commit: robot awesome_leg, 8 links, 7 joints
Links:
- removed link hip1_1
- removed link hip2_1
- removed link knee_1
- added link shank, mass 2.7264471; collision mesh filename=package://awesome_leg/description/meshes/collision/hip-pitc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 scale=0.001 0.001 0.001; visual mesh filename=package://awesome_leg/description/meshes/visual/hip-pitch.s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 scale=0.001 0.001 0.001
- added link shin, mass 1.23787877e+00; collision mesh filename=package://awesome_leg/description/meshes/collision/front_ri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 scale=0.001 0.001 0.001; visual mesh filename=package://awesome_leg/description/meshes/visual/front_right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 scale=0.001 0.001 0.001
- link pelvis: mass 1.0 -> None; geometry 
Joints:
- removed joint hip_yaw_1
- joint hip_pitch_1: child hip2_1 -> shank; origin xyz=0.0 0.0 0.0625 rpy=1.57079632679 0.0 1.5707963268 -> xyz=0.0 0.0 0.0 rpy=-1.57079632679 0 -1.57079632679; parent hip1_1 -> pelvis
- joint knee_pitch_1: child knee_1 -> shin; parent hip2_1 -> shank
- joint test_rig2payload: origin xyz=0.18 0 0.3691 -> xyz=0.18 0 0.25
- joint tip_joint: parent knee_1 -> shin

Commit message: reversed knee joint axis to comply with hw

File: description/urdf/awesome_leg.urdf.xacro (robot description, xacro)
@@ -39,5 +39,5 @@
             <child link="shin${id}"/>
             <origin rpy="0.0 0.0 0.0" xyz="0.0 ${-118.2 * mmTom} ${-300.0 * mmTom}"/>
-            <axis xyz="0 1 0"/>
+            <axis xyz="0 -1 0"/>
             <limit effort="112" lower="-2.4" upper="2.4" velocity="20.0"/>
         </joint>

Commit message: still need to fix seg fault

File: description/urdf/awesome_leg.urdf.xacro (robot description, xacro)
@@ -6,5 +6,5 @@
         <xacro:unless value="${ base_link=='None' or base_link=='none'}">
             <!-- only add joint to base if argument is non-empty -->
-            <joint name="hip_pitch${id}" type="revolute">
+            <joint name="hip_pitch_${id}" type="revolute">
                 <parent link="${base_link}" />
                 <child link="femur${id}" />
@@ -35,5 +35,5 @@
             </collision>
         </link>
-        <joint name="knee_pitch${id}" type="revolute">
+        <joint name="knee_pitch_${id}" type="revolute">
             <parent link="femur${id}"/>
             <child link="shin${id}"/>
@@ -64,5 +64,5 @@
         </link>
         <xacro:unless value="${ add_ft_sensor == True}">
-            <joint name="tip_joint${id}" type="fixed">
+            <joint name="tip_joint_${id}" type="fixed">
                 <parent link="shin${id}"/>
                 <child link="tip${id}"/>
@@ -72,5 +72,5 @@
         </xacro:unless>
         <xacro:if value="${ add_ft_sensor == True}">
-            <joint name="tip_joint${id}" type="prismatic">
+            <joint name="tip_joint_${id}" type="prismatic">
                 <parent link="shin${id}"/>
                 <child link="tip${id}"/>

File: description/urdf/generated/awesome_leg.urdf (robot description, URDF)
Before this commit: robot awesome_leg, 6 links, 5 joints
Joints:
- removed joint hip_pitch1
- removed joint knee_pitch1
- removed joint tip_joint1
- added joint hip_pitch_1: type revolute, parent base_link, child femur1, origin xyz=0 0.21459999999999999 0, axis 0 1 0, limit lower=-2.4 upper=2.4 effort=112 velocity=20.0
- added joint knee_pitch_1: type revolute, parent femur1, child shin1, origin xyz=0.0 -0.1182 -0.3 rpy=0.0 0.0 0.0, axis 0 -1 0, limit lower=-2.4 upper=2.4 effort=112 velocity=20.0
- added joint tip_joint_1: type fixed, parent shin1, child tip1, origin xyz=0.0 0.0233 -0.451

File: description/urdf/generated/awesome_leg_standalone.urdf (robot description, URDF)
Before this commit: robot awesome_leg, 3 links, 2 joints
Joints:
- removed joint knee_pitch1
- removed joint tip_joint1
- added joint knee_pitch_1: type revolute, parent femur1, child shin1, origin xyz=0.0 -0.1182 -0.3 rpy=0.0 0.0 0.0, axis 0 -1 0, limit lower=-2.4 upper=2.4 effort=112 velocity=20.0
- added joint tip_joint_1: type fixed, parent shin1, child tip1, origin xyz=0.0 0.0233 -0.451

File: description/urdf/generated/awesome_leg_xbot.urdf (robot description, URDF)
Before this commit: robot awesome_leg, 5 links, 4 joints
Joints:
- removed joint hip_pitch1
- removed joint knee_pitch1
- removed joint tip_joint1
- added joint hip_pitch_1: type revolute, parent base_link, child femur1, origin xyz=0 0.21459999999999999 0, axis 0 1 0, limit lower=-2.4 upper=2.4 effort=112 velocity=20.0
- added joint knee_pitch_1: type revolute, parent femur1, child shin1, origin xyz=0.0 -0.1182 -0.3 rpy=0.0 0.0 0.0, axis 0 -1 0, limit lower=-2.4 upper=2.4 effort=112 velocity=20.0
- added joint tip_joint_1: type fixed, parent shin1, child tip1, origin xyz=0.0 0.0233 -0.451
