Commit message: still trying to find decent collision params

File: description/urdf/awesome_leg.urdf.xacro (robot description, xacro)
@@ -94,5 +94,23 @@
                             <sphere radius="${fts_sphere_radius}"/>
                         </geometry>
-                        <max_contacts> 20 </max_contacts>
+                        <max_contacts> 1 </max_contacts>
+                        <!-- <surface>
+                            <contact>
+                                <ode>
+                                    <kp>1000000000</kp>
+                                    <kd>1</kd>
+                                    <min_depth> 0 </min_depth>
+                                    <max_vel>0.01</max_vel>-
+                                    <soft_cfm> 0.01 </soft_cfm>
+                                    <soft_erp> 0.2 </soft_erp>
+                                </ode>
+                            </contact>
+                            <friction>
+                                <ode>
+                                <mu>1</mu>
+                                <mu2>1</mu2>
+                                </ode>
+                            </friction>
+                        </surface> -->
                     </collision>
             </link>

File: description/urdf/utils.urdf.xacro (robot description, xacro)
@@ -21,5 +21,5 @@
 <xacro:property name="fts_sphere_radius" value="0.001" />
 <xacro:property name="fts_delta" value="0.000" />
-<xacro:property name="aux_mass_tip" value="0.005" />
+<xacro:property name="aux_mass_tip" value="0.01" />
 <!-- color -->
 <material name="darkblue">

Commit message: fixed missing offsets on inertial frames

File: description/urdf/awesome_leg.urdf.xacro (robot description, xacro)
@@ -16,5 +16,5 @@
         <link name="femur${id}">
             <inertial>
-                <origin xyz="0.0 0.0 0.0"/>
+                <origin rpy="${89.6977809 * DEG2RAD} ${-80.3474629 * DEG2RAD} ${-89.9195968 * DEG2RAD}" xyz="${-1.7807105e-02 * mmTom} ${-3.4271947e+01 * mmTom} ${-2.2282064e+02 * mmTom}"/>
                 <mass value="3.3712777"/>
                 <inertia ixx="${4.6647423e+04 * kgmm2_2_kgm2}" iyy="${4.3720135e+04 * kgmm2_2_kgm2}" izz="${7.5794813e+04 * kgmm2_2_kgm2}"
@@ -44,5 +44,5 @@
         <link name="shin${id}">
             <inertial>
-                <origin xyz="0.0 0.0 0.0"/>
+                <origin rpy="${-87.960 * DEG2RAD} ${0.0 * DEG2RAD} ${-90 * DEG2RAD}" xyz="${9.2284672e-04 * mmTom} ${1.759883e+01 * mmTom} ${-1.8730054e+02 * mmTom}"/>
                 <mass value="1.3106594"/>
                 <inertia ixx="${4.0133965e+04 * kgmm2_2_kgm2}" iyy="${4.0269285e+04 * kgmm2_2_kgm2}" izz="${1.5274496e+03 * kgmm2_2_kgm2}"

File: description/urdf/awesome_leg_test_rig.urdf.xacro (robot description, xacro)
@@ -63,5 +63,5 @@
         </visual>
         <collision>
-            <origin xyz="0.0 0.0 0.0" rpy="0.0 0.0 0.0"/>
+            <origin xyz="0 0 0" rpy="0.0 0.0 0.0"/>
             <geometry>
                 <mesh filename="package://awesome_leg/description/new_meshes/collision/base.stl" scale="${dmTom} ${dmTom} ${dmTom}"/>
@@ -69,5 +69,6 @@
         </collision>
         <inertial>
-            <mass value="${4.5477704 + payload_mass}" />
+            <origin rpy="${89.9076318 * DEG2RAD} ${43.5501361 * DEG2RAD} ${89.8459487 * DEG2RAD}" xyz="${-6.0548104e-03 * mmTom} ${8.2902397e+01 * mmTom} ${6.0505209e+01 * mmTom}"/>
+            <mass value="${7.3800519 + payload_mass}" />
             <inertia ixx="${4.4624842e+04 * kgmm2_2_kgm2}" iyy="${2.6977590e+04 * kgmm2_2_kgm2}" izz="${2.7956754e+04 * kgmm2_2_kgm2}"
                     ixy="${-1.4644878e+01 * kgmm2_2_kgm2}" ixz="${3.0225947e+01 * kgmm2_2_kgm2}" iyz="${9.6636358e+03 * kgmm2_2_kgm2}" />

File: description/urdf/generated/awesome_leg.urdf (robot description, URDF)
Before this commit: robot awesome_leg, 6 links, 5 joints
Links:
- link base_link: mass 6.5477704 -> 7.3800519

File: description/urdf/utils.urdf.xacro (robot description, xacro)
@@ -14,7 +14,7 @@
 <xacro:property name="sliding_guide_dyn_friction" value="0.0" />
 <!--<xacro:property name="sliding_guide_dyn_friction" value="50.0" />-->
-<xacro:property name="base_link_mass_compensation" value="2.0" />
-<xacro:property name="payload_mass" value="${0.0 + base_link_mass_compensation}" />
-<!-- <xacro:property name="payload_mass" value="7.38" /> -->
+<!--<xacro:property name="base_link_mass_compensation" value="2.0" />
+<xacro:property name="payload_mass" value="${0.0 + base_link_mass_compensation}" />-->
+<xacro:property name="payload_mass" value="${0.0}" />
 <xacro:property name="camera_height" value="0.5" />
 <xacro:property name="camera_depth" value="1.0" />

Commit message: removed rotations of inertia frames since not supported by xbot

File: description/urdf/awesome_leg.urdf.xacro (robot description, xacro)
@@ -16,5 +16,5 @@
         <link name="femur${id}">
             <inertial>
-                <origin rpy="${89.6977809 * DEG2RAD} ${-80.3474629 * DEG2RAD} ${-89.9195968 * DEG2RAD}" xyz="${-1.7807105e-02 * mmTom} ${-3.4271947e+01 * mmTom} ${-2.2282064e+02 * mmTom}"/>
+                <origin rpy="${0 * DEG2RAD} ${0 * DEG2RAD} ${0 * DEG2RAD}" xyz="${-1.7807105e-02 * mmTom} ${-3.4271947e+01 * mmTom} ${-2.2282064e+02 * mmTom}"/>
                 <mass value="3.3712777"/>
                 <inertia ixx="${4.6647423e+04 * kgmm2_2_kgm2}" iyy="${4.3720135e+04 * kgmm2_2_kgm2}" izz="${7.5794813e+04 * kgmm2_2_kgm2}"
@@ -44,5 +44,5 @@
         <link name="shin${id}">
             <inertial>
-                <origin rpy="${-87.960 * DEG2RAD} ${0.0 * DEG2RAD} ${-90 * DEG2RAD}" xyz="${9.2284672e-04 * mmTom} ${1.759883e+01 * mmTom} ${-1.8730054e+02 * mmTom}"/>
+                <origin rpy="${0.0 * DEG2RAD} ${0.0 * DEG2RAD} ${0 * DEG2RAD}" xyz="${9.2284672e-04 * mmTom} ${1.759883e+01 * mmTom} ${-1.8730054e+02 * mmTom}"/>
                 <mass value="1.3106594"/>
                 <inertia ixx="${4.0133965e+04 * kgmm2_2_kgm2}" iyy="${4.0269285e+04 * kgmm2_2_kgm2}" izz="${1.5274496e+03 * kgmm2_2_kgm2}"

File: description/urdf/awesome_leg_test_rig.urdf.xacro (robot description, xacro)
@@ -69,5 +69,5 @@
         </collision>
         <inertial>
-            <origin rpy="${89.9076318 * DEG2RAD} ${43.5501361 * DEG2RAD} ${89.8459487 * DEG2RAD}" xyz="${-6.0548104e-03 * mmTom} ${8.2902397e+01 * mmTom} ${6.0505209e+01 * mmTom}"/>
+            <origin rpy="${0 * DEG2RAD} ${0 * DEG2RAD} ${0 * DEG2RAD}" xyz="${-6.0548104e-03 * mmTom} ${8.2902397e+01 * mmTom} ${6.0505209e+01 * mmTom}"/>
             <mass value="${7.3800519 + payload_mass}" />
             <inertia ixx="${4.4624842e+04 * kgmm2_2_kgm2}" iyy="${2.6977590e+04 * kgmm2_2_kgm2}" izz="${2.7956754e+04 * kgmm2_2_kgm2}"
