Commit message: jump server addition and jump optimizer tuning

File: description/urdf/awesome_leg_test_rig.urdf.xacro (robot description, xacro)
@@ -9,5 +9,5 @@
     <xacro:property name="hip_mounting_offset" value="0.08" />
     <xacro:property name="pelvis_mounting_height" value="0.3691" />
-    <xacro:property name="payload_mass" value="10.0" />
+    <xacro:property name="payload_mass" value="4.0" />
     <link name="world" />
     <!-- fixing the test rig to the world -->

File: description/urdf/generated/awesome_leg_test_rig.urdf (robot description, URDF)
Before this commit: robot awesome_leg, 8 links, 7 joints
Links:
- link payload_link: mass 10.0 -> 4.0

Commit message: other jump generation

File: description/urdf/awesome_leg_test_rig.urdf.xacro (robot description, xacro)
@@ -15,5 +15,5 @@
         <xacro:property name="pelvis_mounting_height" value="0.3691" />
     </xacro:unless>
-    <xacro:property name="payload_mass" value="10.0" />
+    <xacro:property name="payload_mass" value="7.38" />
     <link name="world" />
     <!-- fixing the test rig to the world -->

File: description/urdf/generated/awesome_leg_test_rig.urdf (robot description, URDF)
Before this commit: robot awesome_leg, 8 links, 7 joints
Links:
- removed link hip1_1
- removed link hip2_1
- removed link knee_1
- added link shank, mass 2.7264471; collision mesh filename=package://awesome_leg/description/meshes/collision/hip-pitc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 scale=0.001 0.001 0.001; visual mesh filename=package://awesome_leg/description/meshes/visual/hip-pitch.s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 scale=0.001 0.001 0.001
- added link shin, mass 1.23787877e+00; collision mesh filename=package://awesome_leg/description/meshes/collision/front_ri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 scale=0.001 0.001 0.001; visual mesh filename=package://awesome_leg/description/meshes/visual/front_right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 scale=0.001 0.001 0.001
- link payload_link: mass 10.0 -> 7.38
- link pelvis: mass 1.0 -> None; geometry 
Joints:
- removed joint hip_yaw_1
- joint hip_pitch_1: child hip2_1 -> shank; limit lower=-2.4 upper=2.4 effort=112 velocity=20.0 -> lower=-2.0226 upper=2.02748 effort=112 velocity=20.0; origin xyz=0.0 0.0 0.0625 rpy=1.57079632679 0.0 1.5707963268 -> xyz=0.0 0.0 0.0 rpy=-1.57079632679 0 -1.57079632679; parent hip1_1 -> pelvis
- joint knee_pitch_1: child knee_1 -> shin; limit lower=-2.4 upper=2.4 effort=112 velocity=20.0 -> lower=-2.0226 upper=2.02748 effort=112 velocity=20.0; parent hip2_1 -> shank
- joint test_rig2payload: origin xyz=0.18 0 0.3691 -> xyz=0.18 0 0.25
- joint tip_joint: parent knee_1 -> shin

Commit message: mounting offset

File: description/urdf/awesome_leg_test_rig.urdf.xacro (robot description, xacro)
@@ -8,5 +8,5 @@
     <xacro:property name="test_rig_height" value="1.0" />
     <xacro:property name="hip_mounting_offset" value="0.08" />
-    <xacro:property name="pelvis_mounting_height" value="0.0" />
+    <xacro:property name="pelvis_mounting_height" value="0.25" />
     <link name="world" />
     <joint name="world_test_rig" type="fixed">

Commit message: made replayer plugin functional again

File: description/urdf/awesome_leg_test_rig.urdf.xacro (robot description, xacro)
@@ -4,4 +4,5 @@
     <xacro:include filename="$(find awesome_leg)/description/urdf/awesome_leg.xbot.xacro"/>
     <xacro:include filename="$(find awesome_leg)/description/urdf/awesome_leg.urdf.xacro"/>
+    <xacro:include filename="$(find awesome_leg)/description/urdf/test_rig.gazebo.xacro"/>
     <xacro:arg name="sliding_guide" default="true" />
     <xacro:property name="test_rig_base_ext" value="0.1" />

File: description/urdf/awesome_leg_xbot.urdf.xacro (robot description, xacro)
@@ -7,5 +7,12 @@
     <xacro:include filename="$(find awesome_leg)/description/urdf/awesome_leg.xbot.xacro"/>
     <xacro:include filename="$(find awesome_leg)/description/urdf/awesome_leg.urdf.xacro"/>
+    <xacro:include filename="$(find awesome_leg)/description/urdf/test_rig.gazebo.xacro"/>
     <link name="world"> </link>
-    <xacro:awesome_leg id="1" base_link="none"/>
+    <joint name="world2base_joint" type="fixed">
+        <origin xyz="0.0 0.0 0.0" rpy="0.0 0.0 0.0"/>
+        <parent link="world"/>
+        <child link="base_link"/>
+    </joint>
+    <link name="base_link"> </link>
+    <xacro:awesome_leg id="1" base_link="base_link"/>
   </robot>

File: description/urdf/generated/awesome_leg_xbot.urdf (robot description, URDF)
Before this commit: robot awesome_leg, 3 links, 2 joints
Links:
- added link base_link
- added link world
Joints:
- added joint hip_pitch1: type revolute, parent base_link, child femur1, origin xyz=0 0.21459999999999999 0, axis 0 1 0, limit lower=-2.4 upper=2.4 effort=112 velocity=20.0
- added joint world2base_joint: type fixed, parent world, child base_link, origin xyz=0.0 0.0 0.0 rpy=0.0 0.0 0.0

Commit message: removed unnecessary test rig collision

File: description/urdf/awesome_leg_test_rig.urdf.xacro (robot description, xacro)
@@ -42,10 +42,10 @@
             <material name="brown"/>
         </visual>
-        <collision>
+        <!--<collision>
             <origin rpy="0 0 0" xyz="0 0 0" />
             <geometry>
                 <box size="${test_rig_base_ext} ${test_rig_base_ext} ${test_rig_height}" />
             </geometry>
-        </collision>
+        </collision>-->
         <inertial>
             <mass value="1000.0" />

Commit message: removed old comment

File: description/urdf/awesome_leg_test_rig.urdf.xacro (robot description, xacro)
@@ -12,20 +12,4 @@
     <xacro:property name="hip_mounting_offset" value="0.08" />
     <xacro:property name="pelvis_mounting_height" value="0.25" />
-    <!-- <xacro:if value="$(arg dump_video_frames)">
-        <joint name="test_rig_2camera_link" type="fixed">
-        <parent link="test_rig" />
-        <child link="camera_link" />
-        <origin xyz="0 ${camera_depth} ${camera_height}" rpy="0 0 0" />
-        </joint>
-        <link name="camera_link">
-            <visual name="visual">
-            <geometry>
-            <box>
-            <size>0.1 0.1 0.1</size>
-            </box>
-            </geometry>
-            </visual>
-        </link>
-    </xacro:if> -->
     <link name="world" />
     <joint name="world_test_rig" type="fixed">

Commit message: added different hip mounting in case of fixed base

File: description/urdf/awesome_leg_test_rig.urdf.xacro (robot description, xacro)
@@ -11,5 +11,10 @@
     <xacro:property name="test_rig_height" value="1.0" />
     <xacro:property name="hip_mounting_offset" value="0.08" />
-    <xacro:property name="pelvis_mounting_height" value="0.25" />
+    <xacro:if value="$(arg sliding_guide)">
+        <xacro:property name="pelvis_mounting_height" value="0.25" />
+    </xacro:if>
+    <xacro:unless value="$(arg sliding_guide)">
+        <xacro:property name="pelvis_mounting_height" value="0.4" />
+    </xacro:unless>
     <link name="world" />
     <joint name="world_test_rig" type="fixed">
