Commit message: added ft sensor info to data and other improvements

File: description/urdf/awesome_leg.xbot.xacro (robot description, xacro)
@@ -22,4 +22,5 @@
             <links>
                 <link name="base_link"/>
+                <link name="tip1"/>
             </links>
         </plugin>
