Commit message: successful jumps in simulation

File: description/urdf/generated/awesome_leg_test_rig.urdf (robot description, URDF)
Before this commit: robot awesome_leg, 7 links, 6 joints
Links:
- removed link shank
- removed link shin
- added link hip1_1, mass 1.9194403; collision mesh filename=package://awesome_leg/description/meshes/collision/hip-yaw.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 scale=0.001 0.001 0.001; visual mesh filename=package://awesome_leg/description/meshes/visual/hip-yaw.stl scale=0.001 0.001 0.001
- added link hip2_1, mass 2.7264471; collision mesh filename=package://awesome_leg/description/meshes/collision/hip-pitc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 scale=0.001 0.001 0.001; visual mesh filename=package://awesome_leg/description/meshes/visual/hip-pitch.s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 scale=0.001 0.001 0.001
- added link knee_1, mass 1.1927236; collision mesh filename=package://awesome_leg/description/meshes/collision/front_ri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 scale=0.001 0.001 0.001; visual mesh filename=package://awesome_leg/description/meshes/visual/front_right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 scale=0.001 0.001 0.001
- link pelvis: mass None -> 1.0; geometry visual cylinder length=0.1 radius=0.1; visual cylinder length=0.1 radius=0.1
Joints:
- added joint hip_yaw_1: type fixed, parent pelvis, child hip1_1, origin xyz=0.0 -0.0 -0.0566 rpy=3.14159265359 0.0 0.0
- joint hip_pitch_1: child shank -> hip2_1; origin xyz=0.0 0.0 0.0 rpy=-1.57079632679 0 -1.57079632679 -> xyz=0.0 0.0 0.0625 rpy=1.57079632679 0.0 1.5707963268; parent pelvis -> hip1_1
- joint knee_pitch_1: child shin -> knee_1; parent shank -> hip2_1
- joint test_rig2payload: origin xyz=0.18 0 0.25 -> xyz=0.18 0 0.3691
- joint tip_joint: parent shin -> knee_1

Commit message: new jumps resampled at 1 KHz

File: description/urdf/generated/awesome_leg_test_rig.urdf (robot description, URDF)
Before this commit: robot awesome_leg, 7 links, 6 joints
Links:
- removed link shank
- removed link shin
- added link hip1_1, mass 1.9194403; collision mesh filename=package://awesome_leg/description/meshes/collision/hip-yaw.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 scale=0.001 0.001 0.001; visual mesh filename=package://awesome_leg/description/meshes/visual/hip-yaw.stl scale=0.001 0.001 0.001
- added link hip2_1, mass 2.7264471; collision mesh filename=package://awesome_leg/description/meshes/collision/hip-pitc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 scale=0.001 0.001 0.001; visual mesh filename=package://awesome_leg/description/meshes/visual/hip-pitch.s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 scale=0.001 0.001 0.001
- added link knee_1, mass 1.1927236; collision mesh filename=package://awesome_leg/description/meshes/collision/front_ri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 scale=0.001 0.001 0.001; visual mesh filename=package://awesome_leg/description/meshes/visual/front_right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 scale=0.001 0.001 0.001
- link pelvis: mass None -> 1.0; geometry visual cylinder length=0.1 radius=0.1; visual cylinder length=0.1 radius=0.1
Joints:
- added joint hip_yaw_1: type fixed, parent pelvis, child hip1_1, origin xyz=0.0 -0.0 -0.0566 rpy=3.14159265359 0.0 0.0
- joint hip_pitch_1: child shank -> hip2_1; limit lower=-2.0226 upper=2.02748 effort=112 velocity=20.0 -> lower=-2.4 upper=2.4 effort=112 velocity=20.0; origin xyz=0.0 0.0 0.0 rpy=-1.57079632679 0 -1.57079632679 -> xyz=0.0 0.0 0.0625 rpy=1.57079632679 0.0 1.5707963268; parent pelvis -> hip1_1
- joint knee_pitch_1: child shin -> knee_1; limit lower=-2.0226 upper=2.02748 effort=112 velocity=20.0 -> lower=-2.4 upper=2.4 effort=112 velocity=20.0; parent shank -> hip2_1
- joint test_rig2payload: origin xyz=0.18 0 0.25 -> xyz=0.18 0 0.3691
- joint tip_joint: parent shin -> knee_1

Commit message: added velocity limits margins in optimization

File: description/urdf/generated/awesome_leg_test_rig.urdf (robot description, URDF)
Before this commit: robot awesome_leg, 8 links, 7 joints
Links:
- removed link hip1_1
- removed link hip2_1
- removed link knee_1
- added link shank, mass 2.7264471; collision mesh filename=package://awesome_leg/description/meshes/collision/hip-pitc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 scale=0.001 0.001 0.001; visual mesh filename=package://awesome_leg/description/meshes/visual/hip-pitch.s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 scale=0.001 0.001 0.001
- added link shin, mass 1.23787877e+00; collision mesh filename=package://awesome_leg/description/meshes/collision/front_ri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 scale=0.001 0.001 0.001; visual mesh filename=package://awesome_leg/description/meshes/visual/front_right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 scale=0.001 0.001 0.001
- link pelvis: mass 1.0 -> None; geometry 
Joints:
- removed joint hip_yaw_1
- joint hip_pitch_1: child hip2_1 -> shank; limit lower=-2.4 upper=2.4 effort=112 velocity=20.0 -> lower=-2.0226 upper=2.02748 effort=112 velocity=20.0; origin xyz=0.0 0.0 0.0625 rpy=1.57079632679 0.0 1.5707963268 -> xyz=0.0 0.0 0.0 rpy=-1.57079632679 0 -1.57079632679; parent hip1_1 -> pelvis
- joint knee_pitch_1: child knee_1 -> shin; limit lower=-2.4 upper=2.4 effort=112 velocity=20.0 -> lower=-2.0226 upper=2.02748 effort=112 velocity=20.0; parent hip2_1 -> shank
- joint test_rig2payload: origin xyz=0.18 0 0.3691 -> xyz=0.18 0 0.25
- joint tip_joint: parent knee_1 -> shin

Commit message: small changes

File: description/urdf/generated/awesome_leg_test_rig.urdf (robot description, URDF)
Before this commit: robot awesome_leg, 6 links, 5 joints
Joints:
- joint knee_pitch1: axis 0 1 0 -> 0 -1 0
