Commit message: added generation of fixed hip urdf

File: description/urdf/generated/awesome_leg_no_sliding.urdf (robot description, URDF)
Before this commit: robot awesome_leg, 6 links, 5 joints
Joints:
- joint test_rig2base: axis 0 0 1 -> (none); limit lower=-10 upper=10.0 effort=500 velocity=50.0 -> (none); type prismatic -> fixed
