Commit message: updated generated urdfs

File: description/urdf/generated/awesome_leg.urdf (robot description, URDF)
Before this commit: robot awesome_leg, 6 links, 5 joints
Links:
- link tip1: mass 0.1 -> None; geometry 
Joints:
- joint tip_joint1: limit lower=0.0 upper=0.0 effort=0 velocity=0.0 -> (none); origin xyz=0.0 0.0233 -0.40900000000000003 -> xyz=0.0 0.0233 -0.451; type revolute -> fixed

Commit message: small change

File: description/urdf/generated/awesome_leg.urdf (robot description, URDF)
Before this commit: robot awesome_leg, 6 links, 5 joints
Links:
- link test_rig: geometry visual box size=0.1 0.1 1.0

File: description/urdf/generated/awesome_leg_no_sliding.urdf (robot description, URDF)
Before this commit: robot awesome_leg, 6 links, 5 joints
Links:
- link test_rig: geometry visual box size=0.1 0.1 1.0
Joints:
- joint test_rig2base: axis (none) -> 0 0 1; limit (none) -> lower=-10 upper=10.0 effort=500 velocity=50.0; type fixed -> prismatic
