Commit message: added automatic urdf generation upon compilation

File: description/urdf/generated/awesome_leg_floating.urdf (robot description, URDF)
Before this commit: robot awesome_leg, 5 links, 4 joints
Links:
- added link test_rig, mass 1000.0; visual box size=0.1 0.1 1.0
Joints:
- added joint test_rig2base: type prismatic, parent test_rig, child base_link, origin xyz=0.18 0 0.25 rpy=0.0 0.0 -1.57079632679, axis 0 0 1, limit lower=-10 upper=10.0 effort=500 velocity=50.0
- joint world_test_rig: child base_link -> test_rig; origin xyz=0.18 0 0.75 rpy=0.0 0.0 -1.57079632679 -> xyz=0 0 0.5; type floating -> fixed

File: description/urdf/generated/awesome_leg_no_sliding.urdf (robot description, URDF)
Before this commit: robot awesome_leg, 6 links, 5 joints
Joints:
- joint test_rig2base: axis (none) -> 0 0 1; limit (none) -> lower=-10 upper=10.0 effort=500 velocity=50.0; type fixed -> prismatic

Commit message: added more xacro to allow compilation of all urdf in cmakelists with xacro_add_xacro_file

File: description/urdf/generated/awesome_leg_floating.urdf (robot description, URDF)
Before this commit: robot awesome_leg, 6 links, 5 joints
Links:
- removed link test_rig
- link base_link: mass 7.3800519 -> 4.5477704
Joints:
- removed joint test_rig2base
- joint world_test_rig: child test_rig -> base_link; origin xyz=0 0 0.5 -> xyz=0.18 0 0.75 rpy=0.0 0.0 -1.57079632679; type fixed -> floating

File: description/urdf/generated/awesome_leg_no_sliding.urdf (robot description, URDF)
Before this commit: robot awesome_leg, 6 links, 5 joints
Joints:
- joint test_rig2base: axis 0 0 1 -> (none); limit lower=-10 upper=10.0 effort=500 velocity=50.0 -> (none); type prismatic -> fixed
